File: hardware/MOSFETS.sch (KiCad schematic (older format))
At the start: 24 parts

Commit message: Updaated Driver section
Parts:
- D1, D2, D3, D4, D5, D6: value D_Schottky -> B0520LW-7-F
Connections:
- net +V renamed Vbatt
Changed lines of the file:
@@
 LIBS:valves
 LIBS:infineon
+LIBS:bldc_v1-cache
 EELAYER 25 0
 EELAYER END
@@
 Date "2018-03-18"
 Rev "1"
-Comp "Loma Enterprises"
+Comp "Loma Incorporated"
 Comment1 ""
 Comment2 ""
@@
 PhaseA
 Text HLabel 1800 900  0    60   Input ~ 0
-+V
+Vbatt
 Wire Wire Line
 	5050 2900 5050 2250
@@
 P 2150 2250
 F 0 "D1" H 2150 2350 50  0000 C CNN
-F 1 "D_Schottky" H 2150 2150 50  0000 C CNN
+F 1 "B0520LW-7-F" H 2100 2150 50  0000 C CNN
 F 2 "" H 2150 2250 50  0001 C CNN
 F 3 "" H 2150 2250 50  0001 C CNN
@@
 P 2150 3800
 F 0 "D2" H 2150 3900 50  0000 C CNN
-F 1 "D_Schottky" H 2150 3700 50  0000 C CNN
+F 1 "B0520LW-7-F" H 2100 3700 50  0000 C CNN
 F 2 "" H 2150 3800 50  0001 C CNN
 F 3 "" H 2150 3800 50  0001 C CNN
@@
 P 4350 3800
 F 0 "D4" H 4350 3900 50  0000 C CNN
-F 1 "D_Schottky" H 4350 3700 50  0000 C CNN
+F 1 "B0520LW-7-F" H 4300 3700 50  0000 C CNN
 F 2 "" H 4350 3800 50  0001 C CNN
 F 3 "" H 4350 3800 50  0001 C CNN
@@
 P 4350 2250
 F 0 "D3" H 4350 2350 50  0000 C CNN
-F 1 "D_Schottky" H 4350 2150 50  0000 C CNN
+F 1 "B0520LW-7-F" H 4300 2150 50  0000 C CNN
 F 2 "" H 4350 2250 50  0001 C CNN
 F 3 "" H 4350 2250 50  0001 C CNN
@@
 P 6550 3800
 F 0 "D6" H 6550 3900 50  0000 C CNN
-F 1 "D_Schottky" H 6550 3700 50  0000 C CNN
+F 1 "B0520LW-7-F" H 6500 3700 50  0000 C CNN
 F 2 "" H 6550 3800 50  0001 C CNN
 F 3 "" H 6550 3800 50  0001 C CNN
@@
 P 6550 2250
 F 0 "D5" H 6550 2350 50  0000 C CNN
-F 1 "D_Schottky" H 6550 2150 50  0000 C CNN
+F 1 "B0520LW-7-F" H 6500 2150 50  0000 C CNN
 F 2 "" H 6550 2250 50  0001 C CNN
 F 3 "" H 6550 2250 50  0001 C CNN

Commit message: Update gate driver protection
Parts:
- added D10, D11, D12, D7, D8, D9: SMBJ14A-13-F, symbol D_Zener
- added MEAS_FB_A, MEAS_FB_B: AD8418, symbol AD8418
- added R13, R14: 0.001, symbol R
- D1, D2, D3, D4, D5, D6: value B0520LW-7-F -> DFLS1100-7
- R10, R11, R12, R7, R8, R9: value 30k -> 20k
Connections:
- net labels added: +5V, 5V, FB_A, FB_B
- wire segments 62 -> 98
Other:
- moved on the sheet: D3, D4, D5, D6, HS_B, HS_C, LS_B, LS_C, R10, R11, R12, R3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

Commit message: Added power converters
Parts:
- R13, R14: PartNumber (none) -> CSNL2512FT1L00
Connections:
- net labels added: 48v
- net labels removed: Vbatt
Changed lines of the file:
@@
 $Descr A4 11693 8268
 encoding utf-8
-Sheet 3 3
+Sheet 3 4
 Title "MOSFETS"
 Date "2018-03-18"
@@
 PhaseA
 Text HLabel 1800 900  0    60   Input ~ 0
-Vbatt
+48v
 Wire Wire Line
 	6250 2900 6250 2250
@@
 	1    0    0    -1
 $EndComp
-Text HLabel 1100 1250 0    60   Input ~ 0
+Text HLabel 1700 700  0    60   Input ~ 0
 +5V
 Connection ~ 6250 900
-Text Label 1250 1250 0    60   ~ 0
+Text Label 1850 700  0    60   ~ 0
 5V
 Wire Wire Line
-	1100 1250 1250 1250
+	1700 700  1850 700
 $Comp
 L R R13
@@
 F 2 "" V 3680 2400 50  0001 C CNN
 F 3 "" H 3750 2400 50  0001 C CNN
+F 4 "CSNL2512FT1L00 " V 3900 2400 60  0000 C CNN "PartNumber"
 	1    3750 2400
 	0    -1   -1   0
@@
 F 2 "" V 7130 2550 50  0001 C CNN
 F 3 "" H 7200 2550 50  0001 C CNN
+F 4 "CSNL2512FT1L00" V 7350 2550 60  0000 C CNN "PartNumber"
 	1    7200 2550
 	0    -1   -1   0

Commit message: added microcontroller page
Parts:
- R1, R2, R3, R4, R5, R6: PN (none) -> CRM2512-JW-100ELF
- R10, R11, R12, R7, R8, R9: PN (none) -> TNPW120620K0BEEA
Connections:
- net labels removed: +5V
Changed lines of the file:
@@
 LIBS:valves
 LIBS:infineon
+LIBS:crf_1
+LIBS:STM32F4-DISCOVERY-SIMON
+LIBS:bldc_v1-cache
 EELAYER 25 0
 EELAYER END
 $Descr A4 11693 8268
 encoding utf-8
-Sheet 3 4
+Sheet 3 5
 Title "MOSFETS"
 Date "2018-03-18"
@@
 F 2 "" V 2080 2000 50  0001 C CNN
 F 3 "" H 2150 2000 50  0001 C CNN
+F 4 "CRM2512-JW-100ELF " V 2050 1850 60  0000 C CNN "PN"
 	1    2150 2000
 	0    1    1    0
@@
 F 2 "" V 2080 3550 50  0001 C CNN
 F 3 "" H 2150 3550 50  0001 C CNN
+F 4 "CRM2512-JW-100ELF " V 2050 3350 60  0000 C CNN "PN"
 	1    2150 3550
 	0    1    1    0
@@
 F 2 "" V 5480 2000 50  0001 C CNN
 F 3 "" H 5550 2000 50  0001 C CNN
+F 4 "CRM2512-JW-100ELF " V 5450 1850 60  0000 C CNN "PN"
 	1    5550 2000
 	0    1    1    0
@@
 F 2 "" V 5480 3550 50  0001 C CNN
 F 3 "" H 5550 3550 50  0001 C CNN
+F 4 "CRM2512-JW-100ELF " V 5450 3400 60  0000 C CNN "PN"
 	1    5550 3550
 	0    1    1    0
@@
 F 2 "" V 8980 1950 50  0001 C CNN
 F 3 "" H 9050 1950 50  0001 C CNN
+F 4 "CRM2512-JW-100ELF " V 8950 1800 60  0000 C CNN "PN"
 	1    9050 1950
 	0    1    1    0
@@
 F 2 "" V 8980 3500 50  0001 C CNN
 F 3 "" H 9050 3500 50  0001 C CNN
+F 4 "CRM2512-JW-100ELF " V 8950 3350 60  0000 C CNN "PN"
 	1    9050 3500
 	0    1    1    0
@@
 F 2 "" V 2530 2450 50  0001 C CNN
 F 3 "" H 2600 2450 50  0001 C CNN
+F 4 "TNPW120620K0BEEA" V 2600 3150 60  0000 C CNN "PN"
 	1    2600 2450
 	0    -1   -1   0
@@
 F 2 "" V 2530 4000 50  0001 C CNN
 F 3 "" H 2600 4000 50  0001 C CNN
+F 4 "TNPW120620K0BEEA " V 2600 4750 60  0000 C CNN "PN"
 	1    2600 4000
 	0    1    1    0
@@
 F 2 "" V 5930 3950 50  0001 C CNN
 F 3 "" H 6000 3950 50  0001 C CNN
+F 4 "TNPW120620K0BEEA " V 6000 4700 60  0000 C CNN "PN"
 	1    6000 3950
 	0    1    1    0
@@
 F 2 "" V 5930 2400 50  0001 C CNN
 F 3 "" H 6000 2400 50  0001 C CNN
+F 4 "TNPW120620K0BEEA " V 6050 1750 60  0000 C CNN "PN"
 	1    6000 2400
 	0    1    1    0
@@
 F 2 "" V 9430 2350 50  0001 C CNN
 F 3 "" H 9500 2350 50  0001 C CNN
+F 4 "TNPW120620K0BEEA " V 9500 3100 60  0000 C CNN "PN"
 	1    9500 2350
 	0    1    1    0
@@
 F 2 "" V 9430 3900 50  0001 C CNN
 F 3 "" H 9500 3900 50  0001 C CNN
+F 4 "TNPW120620K0BEEA " V 9500 4650 60  0000 C CNN "PN"
 	1    9500 3900
 	0    1    1    0
@@
 $EndComp
 Text HLabel 1700 700  0    60   Input ~ 0
-+5V
+5V
 Connection ~ 6250 900
 Text Label 1850 700  0    60   ~ 0

Commit message: associated footprints
Parts:
- D1, D2, D3, D4, D5, D6: footprint (none) -> Diodes_SMD:D_PowerDI-123
- D10, D11, D12, D7, D8, D9: footprint (none) -> Diodes_SMD:D_2114
- HS_A, HS_B, HS_C, LS_A, LS_B, LS_C: footprint (none) -> TO_SOT_Packages_SMD:TO-263-7_TabPin4
- MEAS_FB_A, MEAS_FB_B: footprint (none) -> Housings_SOIC:SO-8_5.3x6.2mm_Pitch1.27mm
- R1, R13, R14, R2, R3, R4, R5, R6: footprint (none) -> Resistors_SMD:R_2512_HandSoldering
- R10, R11, R12, R7, R8, R9: footprint (none) -> Resistors_SMD:R_1206_HandSoldering
Changed lines of the file:
@@
 F 0 "HS_A" H 2200 2100 60  0000 C CNN
 F 1 "IPB017N10N5" H 2200 2000 60  0000 C CNN
-F 2 "" H 2200 2000 60  0001 C CNN
+F 2 "TO_SOT_Packages_SMD:TO-263-7_TabPin4" H 2200 2000 60  0001 C CNN
 F 3 "" H 2200 2000 60  0001 C CNN
 	1    2850 1800
@@
 F 0 "HS_B" H 5600 2100 60  0000 C CNN
 F 1 "IPB017N10N5" H 5600 2000 60  0000 C CNN
-F 2 "" H 5600 2000 60  0001 C CNN
+F 2 "TO_SOT_Packages_SMD:TO-263-7_TabPin4" H 5600 2000 60  0001 C CNN
 F 3 "" H 5600 2000 60  0001 C CNN
 	1    6250 1800
@@
 F 0 "HS_C" H 9100 2050 60  0000 C CNN
 F 1 "IPB017N10N5" H 9100 1950 60  0000 C CNN
-F 2 "" H 9100 1950 60  0001 C CNN
+F 2 "TO_SOT_Packages_SMD:TO-263-7_TabPin4" H 9100 1950 60  0001 C CNN
 F 3 "" H 9100 1950 60  0001 C CNN
 	1    9750 1750
@@
 F 0 "LS_A" H 2200 3650 60  0000 C CNN
 F 1 "IPB017N10N5" H 2200 3550 60  0000 C CNN
-F 2 "" H 2200 3550 60  0001 C CNN
+F 2 "TO_SOT_Packages_SMD:TO-263-7_TabPin4" H 2200 3550 60  0001 C CNN
 F 3 "" H 2200 3550 60  0001 C CNN
 	1    2850 3350
@@
 F 0 "LS_B" H 5600 3650 60  0000 C CNN
 F 1 "IPB017N10N5" H 5600 3550 60  0000 C CNN
-F 2 "" H 5600 3550 60  0001 C CNN
+F 2 "TO_SOT_Packages_SMD:TO-263-7_TabPin4" H 5600 3550 60  0001 C CNN
 F 3 "" H 5600 3550 60  0001 C CNN
 	1    6250 3350
@@
 F 0 "LS_C" H 9100 3600 60  0000 C CNN
 F 1 "IPB017N10N5" H 9100 3500 60  0000 C CNN
-F 2 "" H 9100 3500 60  0001 C CNN
+F 2 "TO_SOT_Packages_SMD:TO-263-7_TabPin4" H 9100 3500 60  0001 C CNN
 F 3 "" H 9100 3500 60  0001 C CNN
 	1    9750 3300
@@
 F 0 "R1" V 2230 2000 50  0000 C CNN
 F 1 "10" V 2150 2000 50  0000 C CNN
-F 2 "" V 2080 2000 50  0001 C CNN
+F 2 "Resistors_SMD:R_2512_HandSoldering" V 2080 2000 50  0001 C CNN
 F 3 "" H 2150 2000 50  0001 C CNN
 F 4 "CRM2512-JW-100ELF " V 2050 1850 60  0000 C CNN "PN"
@@
 F 0 "R2" V 2230 3550 50  0000 C CNN
 F 1 "10" V 2150 3550 50  0000 C CNN
-F 2 "" V 2080 3550 50  0001 C CNN
+F 2 "Resistors_SMD:R_2512_HandSoldering" V 2080 3550 50  0001 C CNN
 F 3 "" H 2150 3550 50  0001 C CNN
 F 4 "CRM2512-JW-100ELF " V 2050 3350 60  0000 C CNN "PN"
@@
 F 0 "R3" V 5630 2000 50  0000 C CNN
 F 1 "10" V 5550 2000 50  0000 C CNN
-F 2 "" V 5480 2000 50  0001 C CNN
+F 2 "Resistors_SMD:R_2512_HandSoldering" V 5480 2000 50  0001 C CNN
 F 3 "" H 5550 2000 50  0001 C CNN
 F 4 "CRM2512-JW-100ELF " V 5450 1850 60  0000 C CNN "PN"
@@
 F 0 "R4" V 5630 3550 50  0000 C CNN
 F 1 "10" V 5550 3550 50  0000 C CNN
-F 2 "" V 5480 3550 50  0001 C CNN
+F 2 "Resistors_SMD:R_2512_HandSoldering" V 5480 3550 50  0001 C CNN
 F 3 "" H 5550 3550 50  0001 C CNN
 F 4 "CRM2512-JW-100ELF " V 5450 3400 60  0000 C CNN "PN"
@@
 F 0 "R5" V 9130 1950 50  0000 C CNN
 F 1 "10" V 9050 1950 50  0000 C CNN
-F 2 "" V 8980 1950 50  0001 C CNN
+F 2 "Resistors_SMD:R_2512_HandSoldering" V 8980 1950 50  0001 C CNN
 F 3 "" H 9050 1950 50  0001 C CNN
 F 4 "CRM2512-JW-100ELF " V 8950 1800 60  0000 C CNN "PN"
@@
 F 0 "R6" V 9130 3500 50  0000 C CNN
 F 1 "10" V 9050 3500 50  0000 C CNN
-F 2 "" V 8980 3500 50  0001 C CNN
+F 2 "Resistors_SMD:R_2512_HandSoldering" V 8980 3500 50  0001 C CNN
 F 3 "" H 9050 3500 50  0001 C CNN
 F 4 "CRM2512-JW-100ELF " V 8950 3350 60  0000 C CNN "PN"
@@
 F 0 "D1" H 2150 2350 50  0000 C CNN
 F 1 "DFLS1100-7" H 2100 2150 50  0000 C CNN
-F 2 "" H 2150 2250 50  0001 C CNN
+F 2 "Diodes_SMD:D_PowerDI-123" H 2150 2250 50  0001 C CNN
 F 3 "" H 2150 2250 50  0001 C CNN
 	1    2150 2250
@@
 F 0 "D2" H 2150 3900 50  0000 C CNN
 F 1 "DFLS1100-7" H 2100 3700 50  0000 C CNN
-F 2 "" H 2150 3800 50  0001 C CNN
+F 2 "Diodes_SMD:D_PowerDI-123" H 2150 3800 50  0001 C CNN
 F 3 "" H 2150 3800 50  0001 C CNN
 	1    2150 3800
@@
 F 0 "D4" H 5550 3900 50  0000 C CNN
 F 1 "DFLS1100-7" H 5500 3700 50  0000 C CNN
-F 2 "" H 5550 3800 50  0001 C CNN
+F 2 "Diodes_SMD:D_PowerDI-123" H 5550 3800 50  0001 C CNN
 F 3 "" H 5550 3800 50  0001 C CNN
 	1    5550 3800
@@
 F 0 "D3" H 5550 2350 50  0000 C CNN
 F 1 "DFLS1100-7" H 5500 2150 50  0000 C CNN
-F 2 "" H 5550 2250 50  0001 C CNN
+F 2 "Diodes_SMD:D_PowerDI-123" H 5550 2250 50  0001 C CNN
 F 3 "" H 5550 2250 50  0001 C CNN
 	1    5550 2250
@@
 F 0 "D6" H 9050 3850 50  0000 C CNN
 F 1 "DFLS1100-7" H 9000 3650 50  0000 C CNN
-F 2 "" H 9050 3750 50  0001 C CNN
+F 2 "Diodes_SMD:D_PowerDI-123" H 9050 3750 50  0001 C CNN
 F 3 "" H 9050 3750 50  0001 C CNN
 	1    9050 3750
@@
 F 0 "D5" H 9050 2300 50  0000 C CNN
 F 1 "DFLS1100-7" H 9000 2100 50  0000 C CNN
-F 2 "" H 9050 2200 50  0001 C CNN
+F 2 "Diodes_SMD:D_PowerDI-123" H 9050 2200 50  0001 C CNN
 F 3 "" H 9050 2200 50  0001 C CNN
 	1    9050 2200
@@
 F 0 "R7" V 2680 2450 50  0000 C CNN
 F 1 "20k" V 2600 2450 50  0000 C CNN
-F 2 "" V 2530 2450 50  0001 C CNN
+F 2 "Resistors_SMD:R_1206_HandSoldering" V 2530 2450 50  0001 C CNN
 F 3 "" H 2600 2450 50  0001 C CNN
 F 4 "TNPW120620K0BEEA" V 2600 3150 60  0000 C CNN "PN"
@@
 F 0 "R8" V 2680 4000 50  0000 C CNN
 F 1 "20k" V 2600 4000 50  0000 C CNN
-F 2 "" V 2530 4000 50  0001 C CNN
+F 2 "Resistors_SMD:R_1206_HandSoldering" V 2530 4000 50  0001 C CNN
 F 3 "" H 2600 4000 50  0001 C CNN
 F 4 "TNPW120620K0BEEA " V 2600 4750 60  0000 C CNN "PN"
@@
 F 0 "R10" V 6080 3950 50  0000 C CNN
 F 1 "20k" V 6000 3950 50  0000 C CNN
-F 2 "" V 5930 3950 50  0001 C CNN
+F 2 "Resistors_SMD:R_1206_HandSoldering" V 5930 3950 50  0001 C CNN
 F 3 "" H 6000 3950 50  0001 C CNN
 F 4 "TNPW120620K0BEEA " V 6000 4700 60  0000 C CNN "PN"
@@
 F 0 "R9" V 6080 2400 50  0000 C CNN
 F 1 "20k" V 6000 2400 50  0000 C CNN
-F 2 "" V 5930 2400 50  0001 C CNN
+F 2 "Resistors_SMD:R_1206_HandSoldering" V 5930 2400 50  0001 C CNN
 F 3 "" H 6000 2400 50  0001 C CNN
 F 4 "TNPW120620K0BEEA " V 6050 1750 60  0000 C CNN "PN"
@@
 F 0 "R11" V 9580 2350 50  0000 C CNN
 F 1 "20k" V 9500 2350 50  0000 C CNN
-F 2 "" V 9430 2350 50  0001 C CNN
+F 2 "Resistors_SMD:R_1206_HandSoldering" V 9430 2350 50  0001 C CNN
 F 3 "" H 9500 2350 50  0001 C CNN
 F 4 "TNPW120620K0BEEA " V 9500 3100 60  0000 C CNN "PN"
@@
 F 0 "R12" V 9580 3900 50  0000 C CNN
 F 1 "20k" V 9500 3900 50  0000 C CNN
-F 2 "" V 9430 3900 50  0001 C CNN
+F 2 "Resistors_SMD:R_1206_HandSoldering" V 9430 3900 50  0001 C CNN
 F 3 "" H 9500 3900 50  0001 C CNN
 F 4 "TNPW120620K0BEEA " V 9500 4650 60  0000 C CNN "PN"
@@
 F 0 "D7" H 2600 2750 50  0000 C CNN
 F 1 "SMBJ14A-13-F" H 2500 2550 50  0000 C CNN
-F 2 "" H 2600 2650 50  0001 C CNN
+F 2 "Diodes_SMD:D_2114" H 2600 2650 50  0001 C CNN
 F 3 "" H 2600 2650 50  0001 C CNN
 	1    2600 2650
@@
 F 0 "D8" H 2600 4350 50  0000 C CNN
 F 1 "SMBJ14A-13-F" H 2500 4150 50  0000 C CNN
-F 2 "" H 2600 4250 50  0001 C CNN
+F 2 "Diodes_SMD:D_2114" H 2600 4250 50  0001 C CNN
 F 3 "" H 2600 4250 50  0001 C CNN
 	1    2600 4250
@@
 F 0 "D10" H 6000 4300 50  0000 C CNN
 F 1 "SMBJ14A-13-F" H 5900 4100 50  0000 C CNN
-F 2 "" H 6000 4200 50  0001 C CNN
+F 2 "Diodes_SMD:D_2114" H 6000 4200 50  0001 C CNN
 F 3 "" H 6000 4200 50  0001 C CNN
 	1    6000 4200
@@
 F 0 "D9" H 6000 2750 50  0000 C CNN
 F 1 "SMBJ14A-13-F" H 5900 2550 50  0000 C CNN
-F 2 "" H 6000 2650 50  0001 C CNN
+F 2 "Diodes_SMD:D_2114" H 6000 2650 50  0001 C CNN
 F 3 "" H 6000 2650 50  0001 C CNN
 	1    6000 2650
@@
 F 0 "D11" H 9500 2700 50  0000 C CNN
 F 1 "SMBJ14A-13-F" H 9400 2500 50  0000 C CNN
-F 2 "" H 9500 2600 50  0001 C CNN
+F 2 "Diodes_SMD:D_2114" H 9500 2600 50  0001 C CNN
 F 3 "" H 9500 2600 50  0001 C CNN
 	1    9500 2600
@@
 F 0 "D12" H 9500 4250 50  0000 C CNN
 F 1 "SMBJ14A-13-F" H 9400 4050 50  0000 C CNN
-F 2 "" H 9500 4150 50  0001 C CNN
+F 2 "Diodes_SMD:D_2114" H 9500 4150 50  0001 C CNN
 F 3 "" H 9500 4150 50  0001 C CNN
 	1    9500 4150
@@
 F 0 "MEAS_FB_A" H 3450 3325 50  0000 R CNN
 F 1 "AD8418" H 3450 3250 50  0000 R CNN
-F 2 "" H 3800 2550 50  0001 C CNN
+F 2 "Housings_SOIC:SO-8_5.3x6.2mm_Pitch1.27mm" H 3800 2550 50  0001 C CNN
 F 3 "" H 4400 2200 50  0001 C CNN
 	1    3750 2900
@@
 F 0 "R13" V 3830 2400 50  0000 C CNN
 F 1 "0.001" V 3750 2400 50  0000 C CNN
-F 2 "" V 3680 2400 50  0001 C CNN
+F 2 "Resistors_SMD:R_2512_HandSoldering" V 3680 2400 50  0001 C CNN
 F 3 "" H 3750 2400 50  0001 C CNN
 F 4 "CSNL2512FT1L00 " V 3900 2400 60  0000 C CNN "PartNumber"
@@
 F 0 "MEAS_FB_B" H 6900 3475 50  0000 R CNN
 F 1 "AD8418" H 6900 3400 50  0000 R CNN
-F 2 "" H 7250 2700 50  0001 C CNN
+F 2 "Housings_SOIC:SO-8_5.3x6.2mm_Pitch1.27mm" H 7250 2700 50  0001 C CNN
 F 3 "" H 7850 2350 50  0001 C CNN
 	1    7200 3050
@@
 F 0 "R14" V 7280 2550 50  0000 C CNN
 F 1 "0.001" V 7200 2550 50  0000 C CNN
-F 2 "" V 7130 2550 50  0001 C CNN
+F 2 "Resistors_SMD:R_2512_HandSoldering" V 7130 2550 50  0001 C CNN
 F 3 "" H 7200 2550 50  0001 C CNN
 F 4 "CSNL2512FT1L00" V 7350 2550 60  0000 C CNN "PartNumber"

Commit message: annotated schematic
Parts:
- renumbered D6 to D10, D7 to D3, D8 to D4, D3 to D5, D4 to D6, D9 to D7, D10 to D8, D5 to D9, HS_A to HS_A1, HS_B to HS_B1, HS_C to HS_C1, LS_A to LS_A1, LS_B to LS_B1, LS_C to LS_C1, MEAS_FB_A to MEAS_FB_A1, MEAS_FB_B to MEAS_FB_B1, R14 to R11, R5 to R12, R6 to R13, R11 to R14, R12 to R15, R1 to R2, R2 to R3, R7 to R4, R8 to R5, R13 to R6, R3 to R7, R4 to R8
Changed lines of the file:
@@
 $EndDescr
 $Comp
-L IPB017N10N5 HS_A
+L IPB017N10N5 HS_A1
 U 1 1 5AAE8FFF
 P 2850 1800
-F 0 "HS_A" H 2200 2100 60  0000 C CNN
+F 0 "HS_A1" H 2200 2100 60  0000 C CNN
 F 1 "IPB017N10N5" H 2200 2000 60  0000 C CNN
 F 2 "TO_SOT_Packages_SMD:TO-263-7_TabPin4" H 2200 2000 60  0001 C CNN
@@
 $EndComp
 $Comp
-L IPB017N10N5 HS_B
+L IPB017N10N5 HS_B1
 U 1 1 5AAE909A
 P 6250 1800
-F 0 "HS_B" H 5600 2100 60  0000 C CNN
+F 0 "HS_B1" H 5600 2100 60  0000 C CNN
 F 1 "IPB017N10N5" H 5600 2000 60  0000 C CNN
 F 2 "TO_SOT_Packages_SMD:TO-263-7_TabPin4" H 5600 2000 60  0001 C CNN
@@
 $EndComp
 $Comp
-L IPB017N10N5 HS_C
+L IPB017N10N5 HS_C1
 U 1 1 5AAE910F
 P 9750 1750
-F 0 "HS_C" H 9100 2050 60  0000 C CNN
+F 0 "HS_C1" H 9100 2050 60  0000 C CNN
 F 1 "IPB017N10N5" H 9100 1950 60  0000 C CNN
 F 2 "TO_SOT_Packages_SMD:TO-263-7_TabPin4" H 9100 1950 60  0001 C CNN
@@
 $EndComp
 $Comp
-L IPB017N10N5 LS_A
+L IPB017N10N5 LS_A1
 U 1 1 5AAE9174
 P 2850 3350
-F 0 "LS_A" H 2200 3650 60  0000 C CNN
+F 0 "LS_A1" H 2200 3650 60  0000 C CNN
 F 1 "IPB017N10N5" H 2200 3550 60  0000 C CNN
 F 2 "TO_SOT_Packages_SMD:TO-263-7_TabPin4" H 2200 3550 60  0001 C CNN
@@
 $EndComp
 $Comp
-L IPB017N10N5 LS_B
+L IPB017N10N5 LS_B1
 U 1 1 5AAE9213
 P 6250 3350
-F 0 "LS_B" H 5600 3650 60  0000 C CNN
+F 0 "LS_B1" H 5600 3650 60  0000 C CNN
 F 1 "IPB017N10N5" H 5600 3550 60  0000 C CNN
 F 2 "TO_SOT_Packages_SMD:TO-263-7_TabPin4" H 5600 3550 60  0001 C CNN
@@
 $EndComp
 $Comp
-L IPB017N10N5 LS_C
+L IPB017N10N5 LS_C1
 U 1 1 5AAE9276
 P 9750 3300
-F 0 "LS_C" H 9100 3600 60  0000 C CNN
+F 0 "LS_C1" H 9100 3600 60  0000 C CNN
 F 1 "IPB017N10N5" H 9100 3500 60  0000 C CNN
 F 2 "TO_SOT_Packages_SMD:TO-263-7_TabPin4" H 9100 3500 60  0001 C CNN
@@
 LS_C_GATE
 $Comp
-L R R1
+L R R2
 U 1 1 5AAEA2F9
 P 2150 2000
-F 0 "R1" V 2230 2000 50  0000 C CNN
+F 0 "R2" V 2230 2000 50  0000 C CNN
 F 1 "10" V 2150 2000 50  0000 C CNN
 F 2 "Resistors_SMD:R_2512_HandSoldering" V 2080 2000 50  0001 C CNN
@@
 $EndComp
 $Comp
-L R R2
+L R R3
 U 1 1 5AAEA36D
 P 2150 3550
-F 0 "R2" V 2230 3550 50  0000 C CNN
+F 0 "R3" V 2230 3550 50  0000 C CNN
 F 1 "10" V 2150 3550 50  0000 C CNN
 F 2 "Resistors_SMD:R_2512_HandSoldering" V 2080 3550 50  0001 C CNN
@@
 $EndComp
 $Comp
-L R R3
+L R R7
 U 1 1 5AAEA3DA
 P 5550 2000
-F 0 "R3" V 5630 2000 50  0000 C CNN
+F 0 "R7" V 5630 2000 50  0000 C CNN
 F 1 "10" V 5550 2000 50  0000 C CNN
 F 2 "Resistors_SMD:R_2512_HandSoldering" V 5480 2000 50  0001 C CNN
@@
 $EndComp
 $Comp
-L R R4
+L R R8
 U 1 1 5AAEA449
 P 5550 3550
-F 0 "R4" V 5630 3550 50  0000 C CNN
+F 0 "R8" V 5630 3550 50  0000 C CNN
 F 1 "10" V 5550 3550 50  0000 C CNN
 F 2 "Resistors_SMD:R_2512_HandSoldering" V 5480 3550 50  0001 C CNN
@@
 $EndComp
 $Comp
-L R R5
+L R R12
 U 1 1 5AAEA476
 P 9050 1950
-F 0 "R5" V 9130 1950 50  0000 C CNN
+F 0 "R12" V 9130 1950 50  0000 C CNN
 F 1 "10" V 9050 1950 50  0000 C CNN
 F 2 "Resistors_SMD:R_2512_HandSoldering" V 8980 1950 50  0001 C CNN
@@
 $EndComp
 $Comp
-L R R6
+L R R13
 U 1 1 5AAEA4AC
 P 9050 3500
-F 0 "R6" V 9130 3500 50  0000 C CNN
+F 0 "R13" V 9130 3500 50  0000 C CNN
 F 1 "10" V 9050 3500 50  0000 C CNN
 F 2 "Resistors_SMD:R_2512_HandSoldering" V 8980 3500 50  0001 C CNN
@@
 $EndComp
 $Comp
-L D_Schottky D4
+L D_Schottky D6
 U 1 1 5AAEB1CB
 P 5550 3800
-F 0 "D4" H 5550 3900 50  0000 C CNN
+F 0 "D6" H 5550 3900 50  0000 C CNN
 F 1 "DFLS1100-7" H 5500 3700 50  0000 C CNN
 F 2 "Diodes_SMD:D_PowerDI-123" H 5550 3800 50  0001 C CNN
@@
 $EndComp
 $Comp
-L D_Schottky D3
+L D_Schottky D5
 U 1 1 5AAEB238
 P 5550 2250
-F 0 "D3" H 5550 2350 50  0000 C CNN
+F 0 "D5" H 5550 2350 50  0000 C CNN
 F 1 "DFLS1100-7" H 5500 2150 50  0000 C CNN
 F 2 "Diodes_SMD:D_PowerDI-123" H 5550 2250 50  0001 C CNN
@@
 $EndComp
 $Comp
-L D_Schottky D6
+L D_Schottky D10
 U 1 1 5AAEB354
 P 9050 3750
-F 0 "D6" H 9050 3850 50  0000 C CNN
+F 0 "D10" H 9050 3850 50  0000 C CNN
 F 1 "DFLS1100-7" H 9000 3650 50  0000 C CNN
 F 2 "Diodes_SMD:D_PowerDI-123" H 9050 3750 50  0001 C CNN
@@
 $EndComp
 $Comp
-L D_Schottky D5
+L D_Schottky D9
 U 1 1 5AAEB3CD
 P 9050 2200
-F 0 "D5" H 9050 2300 50  0000 C CNN
+F 0 "D9" H 9050 2300 50  0000 C CNN
 F 1 "DFLS1100-7" H 9000 2100 50  0000 C CNN
 F 2 "Diodes_SMD:D_PowerDI-123" H 9050 2200 50  0001 C CNN
@@
 $EndComp
 $Comp
-L R R7
+L R R4
 U 1 1 5AAEB875
 P 2600 2450
-F 0 "R7" V 2680 2450 50  0000 C CNN
+F 0 "R4" V 2680 2450 50  0000 C CNN
 F 1 "20k" V 2600 2450 50  0000 C CNN
 F 2 "Resistors_SMD:R_1206_HandSoldering" V 2530 2450 50  0001 C CNN
@@
 Connection ~ 2400 2250
 $Comp
-L R R8
+L R R5
 U 1 1 5AAEBFF4
 P 2600 4000
-F 0 "R8" V 2680 4000 50  0000 C CNN
+F 0 "R5" V 2680 4000 50  0000 C CNN
 F 1 "20k" V 2600 4000 50  0000 C CNN
 F 2 "Resistors_SMD:R_1206_HandSoldering" V 2530 4000 50  0001 C CNN
@@
 Connection ~ 9300 1950
 $Comp
-L R R11
+L R R14
 U 1 1 5AAECB0F
 P 9500 2350
-F 0 "R11" V 9580 2350 50  0000 C CNN
+F 0 "R14" V 9580 2350 50  0000 C CNN
 F 1 "20k" V 9500 2350 50  0000 C CNN
 F 2 "Resistors_SMD:R_1206_HandSoldering" V 9430 2350 50  0001 C CNN
@@
 Connection ~ 9300 3500
 $Comp
-L R R12
+L R R15
 U 1 1 5AAECEF5
 P 9500 3900
-F 0 "R12" V 9580 3900 50  0000 C CNN
+F 0 "R15" V 9580 3900 50  0000 C CNN
 F 1 "20k" V 9500 3900 50  0000 C CNN
 F 2 "Resistors_SMD:R_1206_HandSoldering" V 9430 3900 50  0001 C CNN
@@
 Connection ~ 2850 2650
 $Comp
-L D_Zener D7
+L D_Zener D3
 U 1 1 5AB071F9
 P 2600 2650
-F 0 "D7" H 2600 2750 50  0000 C CNN
+F 0 "D3" H 2600 2750 50  0000 C CNN
 F 1 "SMBJ14A-13-F" H 2500 2550 50  0000 C CNN
 F 2 "Diodes_SMD:D_2114" H 2600 2650 50  0001 C CNN
@@
 $EndComp
 $Comp
-L D_Zener D8
+L D_Zener D4
 U 1 1 5AB07384
 P 2600 4250
-F 0 "D8" H 2600 4350 50  0000 C CNN
+F 0 "D4" H 2600 4350 50  0000 C CNN
 F 1 "SMBJ14A-13-F" H 2500 4150 50  0000 C CNN
 F 2 "Diodes_SMD:D_2114" H 2600 4250 50  0001 C CNN
@@
 Connection ~ 2400 4000
 $Comp
-L D_Zener D10
+L D_Zener D8
 U 1 1 5AB076A1
 P 6000 4200
-F 0 "D10" H 6000 4300 50  0000 C CNN
+F 0 "D8" H 6000 4300 50  0000 C CNN
 F 1 "SMBJ14A-13-F" H 5900 4100 50  0000 C CNN
 F 2 "Diodes_SMD:D_2114" H 6000 4200 50  0001 C CNN
@@
 Connection ~ 5800 3950
 $Comp
-L D_Zener D9
+L D_Zener D7
 U 1 1 5AB0789C
 P 6000 2650
-F 0 "D9" H 6000 2750 50  0000 C CNN
+F 0 "D7" H 6000 2750 50  0000 C CNN
 F 1 "SMBJ14A-13-F" H 5900 2550 50  0000 C CNN
 F 2 "Diodes_SMD:D_2114" H 6000 2650 50  0001 C CNN
@@
 Connection ~ 9300 3900
 $Comp
-L AD8418 MEAS_FB_A
+L AD8418 MEAS_FB_A1
 U 1 1 5AB0952B
 P 3750 2900
-F 0 "MEAS_FB_A" H 3450 3325 50  0000 R CNN
+F 0 "MEAS_FB_A1" H 3450 3325 50  0000 R CNN
 F 1 "AD8418" H 3450 3250 50  0000 R CNN
 F 2 "Housings_SOIC:SO-8_5.3x6.2mm_Pitch1.27mm" H 3800 2550 50  0001 C CNN
@@
 	1700 700  1850 700
 $Comp
-L R R13
+L R R6
 U 1 1 5AB0B7A4
 P 3750 2400
-F 0 "R13" V 3830 2400 50  0000 C CNN
+F 0 "R6" V 3830 2400 50  0000 C CNN
 F 1 "0.001" V 3750 2400 50  0000 C CNN
 F 2 "Resistors_SMD:R_2512_HandSoldering" V 3680 2400 50  0001 C CNN
@@
 Connection ~ 3550 2400
 $Comp
-L AD8418 MEAS_FB_B
+L AD8418 MEAS_FB_B1
 U 1 1 5AB0D80F
 P 7200 3050
-F 0 "MEAS_FB_B" H 6900 3475 50  0000 R CNN
+F 0 "MEAS_FB_B1" H 6900 3475 50  0000 R CNN
 F 1 "AD8418" H 6900 3400 50  0000 R CNN
 F 2 "Housings_SOIC:SO-8_5.3x6.2mm_Pitch1.27mm" H 7250 2700 50  0001 C CNN
@@
 $EndComp
 $Comp
-L R R14
+L R R11
 U 1 1 5AB0D8B6
 P 7200 2550
-F 0 "R14" V 7280 2550 50  0000 C CNN
+F 0 "R11" V 7280 2550 50  0000 C CNN
 F 1 "0.001" V 7200 2550 50  0000 C CNN
 F 2 "Resistors_SMD:R_2512_HandSoldering" V 7130 2550 50  0001 C CNN
