File: hardware/MOSFETS.sch (KiCad schematic (older format))
At the start: 34 parts

Commit message: created new footprints, modified schematic
Parts:
- renumbered HS_A1 to M1, LS_A1 to M2, HS_B1 to M3, LS_B1 to M4, HS_C1 to M5, LS_C1 to M6, R2 to R1, R11 to R10, R12 to R11, R13 to R12, R14 to R13, R15 to R14, R3 to R2, R4 to R3, R5 to R4, R6 to R5, R7 to R6, R8 to R7, R9 to R8, R10 to R9, MEAS_FB_A1 to U1, MEAS_FB_B1 to U2
Changed lines of the file:
@@
 $EndDescr
 $Comp
-L IPB017N10N5 HS_A1
+L IPB017N10N5 M1
 U 1 1 5AAE8FFF
 P 2850 1800
-F 0 "HS_A1" H 2200 2100 60  0000 C CNN
+F 0 "M1" H 2200 2100 60  0000 C CNN
 F 1 "IPB017N10N5" H 2200 2000 60  0000 C CNN
 F 2 "TO_SOT_Packages_SMD:TO-263-7_TabPin4" H 2200 2000 60  0001 C CNN
@@
 $EndComp
 $Comp
-L IPB017N10N5 HS_B1
+L IPB017N10N5 M3
 U 1 1 5AAE909A
 P 6250 1800
-F 0 "HS_B1" H 5600 2100 60  0000 C CNN
+F 0 "M3" H 5600 2100 60  0000 C CNN
 F 1 "IPB017N10N5" H 5600 2000 60  0000 C CNN
 F 2 "TO_SOT_Packages_SMD:TO-263-7_TabPin4" H 5600 2000 60  0001 C CNN
@@
 $EndComp
 $Comp
-L IPB017N10N5 HS_C1
+L IPB017N10N5 M5
 U 1 1 5AAE910F
 P 9750 1750
-F 0 "HS_C1" H 9100 2050 60  0000 C CNN
+F 0 "M5" H 9100 2050 60  0000 C CNN
 F 1 "IPB017N10N5" H 9100 1950 60  0000 C CNN
 F 2 "TO_SOT_Packages_SMD:TO-263-7_TabPin4" H 9100 1950 60  0001 C CNN
@@
 $EndComp
 $Comp
-L IPB017N10N5 LS_A1
+L IPB017N10N5 M2
 U 1 1 5AAE9174
 P 2850 3350
-F 0 "LS_A1" H 2200 3650 60  0000 C CNN
+F 0 "M2" H 2200 3650 60  0000 C CNN
 F 1 "IPB017N10N5" H 2200 3550 60  0000 C CNN
 F 2 "TO_SOT_Packages_SMD:TO-263-7_TabPin4" H 2200 3550 60  0001 C CNN
@@
 $EndComp
 $Comp
-L IPB017N10N5 LS_B1
+L IPB017N10N5 M4
 U 1 1 5AAE9213
 P 6250 3350
-F 0 "LS_B1" H 5600 3650 60  0000 C CNN
+F 0 "M4" H 5600 3650 60  0000 C CNN
 F 1 "IPB017N10N5" H 5600 3550 60  0000 C CNN
 F 2 "TO_SOT_Packages_SMD:TO-263-7_TabPin4" H 5600 3550 60  0001 C CNN
@@
 $EndComp
 $Comp
-L IPB017N10N5 LS_C1
+L IPB017N10N5 M6
 U 1 1 5AAE9276
 P 9750 3300
-F 0 "LS_C1" H 9100 3600 60  0000 C CNN
+F 0 "M6" H 9100 3600 60  0000 C CNN
 F 1 "IPB017N10N5" H 9100 3500 60  0000 C CNN
 F 2 "TO_SOT_Packages_SMD:TO-263-7_TabPin4" H 9100 3500 60  0001 C CNN
@@
 LS_C_GATE
 $Comp
-L R R2
+L R R1
 U 1 1 5AAEA2F9
 P 2150 2000
-F 0 "R2" V 2230 2000 50  0000 C CNN
+F 0 "R1" V 2230 2000 50  0000 C CNN
 F 1 "10" V 2150 2000 50  0000 C CNN
 F 2 "Resistors_SMD:R_2512_HandSoldering" V 2080 2000 50  0001 C CNN
@@
 $EndComp
 $Comp
-L R R3
+L R R2
 U 1 1 5AAEA36D
 P 2150 3550
-F 0 "R3" V 2230 3550 50  0000 C CNN
+F 0 "R2" V 2230 3550 50  0000 C CNN
 F 1 "10" V 2150 3550 50  0000 C CNN
 F 2 "Resistors_SMD:R_2512_HandSoldering" V 2080 3550 50  0001 C CNN
@@
 $EndComp
 $Comp
-L R R7
+L R R6
 U 1 1 5AAEA3DA
 P 5550 2000
-F 0 "R7" V 5630 2000 50  0000 C CNN
+F 0 "R6" V 5630 2000 50  0000 C CNN
 F 1 "10" V 5550 2000 50  0000 C CNN
 F 2 "Resistors_SMD:R_2512_HandSoldering" V 5480 2000 50  0001 C CNN
@@
 $EndComp
 $Comp
-L R R8
+L R R7
 U 1 1 5AAEA449
 P 5550 3550
-F 0 "R8" V 5630 3550 50  0000 C CNN
+F 0 "R7" V 5630 3550 50  0000 C CNN
 F 1 "10" V 5550 3550 50  0000 C CNN
 F 2 "Resistors_SMD:R_2512_HandSoldering" V 5480 3550 50  0001 C CNN
@@
 $EndComp
 $Comp
-L R R12
+L R R11
 U 1 1 5AAEA476
 P 9050 1950
-F 0 "R12" V 9130 1950 50  0000 C CNN
+F 0 "R11" V 9130 1950 50  0000 C CNN
 F 1 "10" V 9050 1950 50  0000 C CNN
 F 2 "Resistors_SMD:R_2512_HandSoldering" V 8980 1950 50  0001 C CNN
@@
 $EndComp
 $Comp
-L R R13
+L R R12
 U 1 1 5AAEA4AC
 P 9050 3500
-F 0 "R13" V 9130 3500 50  0000 C CNN
+F 0 "R12" V 9130 3500 50  0000 C CNN
 F 1 "10" V 9050 3500 50  0000 C CNN
 F 2 "Resistors_SMD:R_2512_HandSoldering" V 8980 3500 50  0001 C CNN
@@
 $EndComp
 $Comp
-L R R4
+L R R3
 U 1 1 5AAEB875
 P 2600 2450
-F 0 "R4" V 2680 2450 50  0000 C CNN
+F 0 "R3" V 2680 2450 50  0000 C CNN
 F 1 "20k" V 2600 2450 50  0000 C CNN
 F 2 "Resistors_SMD:R_1206_HandSoldering" V 2530 2450 50  0001 C CNN
@@
 Connection ~ 2400 2250
 $Comp
-L R R5
+L R R4
 U 1 1 5AAEBFF4
 P 2600 4000
-F 0 "R5" V 2680 4000 50  0000 C CNN
+F 0 "R4" V 2680 4000 50  0000 C CNN
 F 1 "20k" V 2600 4000 50  0000 C CNN
 F 2 "Resistors_SMD:R_1206_HandSoldering" V 2530 4000 50  0001 C CNN
@@
 Connection ~ 5800 3550
 $Comp
-L R R10
+L R R9
 U 1 1 5AAEC38A
 P 6000 3950
-F 0 "R10" V 6080 3950 50  0000 C CNN
+F 0 "R9" V 6080 3950 50  0000 C CNN
 F 1 "20k" V 6000 3950 50  0000 C CNN
 F 2 "Resistors_SMD:R_1206_HandSoldering" V 5930 3950 50  0001 C CNN
@@
 Connection ~ 5800 2000
 $Comp
-L R R9
+L R R8
 U 1 1 5AAEC68E
 P 6000 2400
-F 0 "R9" V 6080 2400 50  0000 C CNN
+F 0 "R8" V 6080 2400 50  0000 C CNN
 F 1 "20k" V 6000 2400 50  0000 C CNN
 F 2 "Resistors_SMD:R_1206_HandSoldering" V 5930 2400 50  0001 C CNN
@@
 Connection ~ 9300 1950
 $Comp
-L R R14
+L R R13
 U 1 1 5AAECB0F
 P 9500 2350
-F 0 "R14" V 9580 2350 50  0000 C CNN
+F 0 "R13" V 9580 2350 50  0000 C CNN
 F 1 "20k" V 9500 2350 50  0000 C CNN
 F 2 "Resistors_SMD:R_1206_HandSoldering" V 9430 2350 50  0001 C CNN
@@
 Connection ~ 9300 3500
 $Comp
-L R R15
+L R R14
 U 1 1 5AAECEF5
 P 9500 3900
-F 0 "R15" V 9580 3900 50  0000 C CNN
+F 0 "R14" V 9580 3900 50  0000 C CNN
 F 1 "20k" V 9500 3900 50  0000 C CNN
 F 2 "Resistors_SMD:R_1206_HandSoldering" V 9430 3900 50  0001 C CNN
@@
 Connection ~ 9300 3900
 $Comp
-L AD8418 MEAS_FB_A1
+L AD8418 U1
 U 1 1 5AB0952B
 P 3750 2900
-F 0 "MEAS_FB_A1" H 3450 3325 50  0000 R CNN
+F 0 "U1" H 3450 3325 50  0000 R CNN
 F 1 "AD8418" H 3450 3250 50  0000 R CNN
 F 2 "Housings_SOIC:SO-8_5.3x6.2mm_Pitch1.27mm" H 3800 2550 50  0001 C CNN
@@
 	1700 700  1850 700
 $Comp
-L R R6
+L R R5
 U 1 1 5AB0B7A4
 P 3750 2400
-F 0 "R6" V 3830 2400 50  0000 C CNN
+F 0 "R5" V 3830 2400 50  0000 C CNN
 F 1 "0.001" V 3750 2400 50  0000 C CNN
 F 2 "Resistors_SMD:R_2512_HandSoldering" V 3680 2400 50  0001 C CNN
@@
 Connection ~ 3550 2400
 $Comp
-L AD8418 MEAS_FB_B1
+L AD8418 U2
 U 1 1 5AB0D80F
 P 7200 3050
-F 0 "MEAS_FB_B1" H 6900 3475 50  0000 R CNN
+F 0 "U2" H 6900 3475 50  0000 R CNN
 F 1 "AD8418" H 6900 3400 50  0000 R CNN
 F 2 "Housings_SOIC:SO-8_5.3x6.2mm_Pitch1.27mm" H 7250 2700 50  0001 C CNN
@@
 $EndComp
 $Comp
-L R R11
+L R R10
 U 1 1 5AB0D8B6
 P 7200 2550
-F 0 "R11" V 7280 2550 50  0000 C CNN
+F 0 "R10" V 7280 2550 50  0000 C CNN
 F 1 "0.001" V 7200 2550 50  0000 C CNN
 F 2 "Resistors_SMD:R_2512_HandSoldering" V 7130 2550 50  0001 C CNN
