File: hardware/MOSFETS.sch (KiCad schematic (older format))
At the start: 34 parts, among them M1 IPB017N10N5, M2 IPB017N10N5, M3 IPB017N10N5, M4 IPB017N10N5, M5 IPB017N10N5, M6 IPB017N10N5, U1 AD8418, U2 AD8418

Commit message: updated part numbers
Parts:
- M1, M2, M3, M4, M5, M6: value IPB017N10N5 -> IPB044N15N5
- U1, U2: value AD8418 -> AD8205
Connections:
- net labels added: PhaseADrain, PhaseBDrain
- wire segments 98 -> 100
Changed lines of the file:
@@
 LIBS:crf_1
 LIBS:STM32F4-DISCOVERY-SIMON
+LIBS:bldc_v1-cache
 EELAYER 25 0
 EELAYER END
@@
 P 2850 1800
 F 0 "M1" H 2200 2100 60  0000 C CNN
-F 1 "IPB017N10N5" H 2200 2000 60  0000 C CNN
+F 1 "IPB044N15N5" H 2200 2000 60  0000 C CNN
 F 2 "TO_SOT_Packages_SMD:TO-263-7_TabPin4" H 2200 2000 60  0001 C CNN
 F 3 "" H 2200 2000 60  0001 C CNN
@@
 P 6250 1800
 F 0 "M3" H 5600 2100 60  0000 C CNN
-F 1 "IPB017N10N5" H 5600 2000 60  0000 C CNN
+F 1 "IPB044N15N5" H 5600 2000 60  0000 C CNN
 F 2 "TO_SOT_Packages_SMD:TO-263-7_TabPin4" H 5600 2000 60  0001 C CNN
 F 3 "" H 5600 2000 60  0001 C CNN
@@
 P 9750 1750
 F 0 "M5" H 9100 2050 60  0000 C CNN
-F 1 "IPB017N10N5" H 9100 1950 60  0000 C CNN
+F 1 "IPB044N15N5" H 9100 1950 60  0000 C CNN
 F 2 "TO_SOT_Packages_SMD:TO-263-7_TabPin4" H 9100 1950 60  0001 C CNN
 F 3 "" H 9100 1950 60  0001 C CNN
@@
 P 2850 3350
 F 0 "M2" H 2200 3650 60  0000 C CNN
-F 1 "IPB017N10N5" H 2200 3550 60  0000 C CNN
+F 1 "IPB044N15N5" H 2200 3550 60  0000 C CNN
 F 2 "TO_SOT_Packages_SMD:TO-263-7_TabPin4" H 2200 3550 60  0001 C CNN
 F 3 "" H 2200 3550 60  0001 C CNN
@@
 P 6250 3350
 F 0 "M4" H 5600 3650 60  0000 C CNN
-F 1 "IPB017N10N5" H 5600 3550 60  0000 C CNN
+F 1 "IPB044N15N5" H 5600 3550 60  0000 C CNN
 F 2 "TO_SOT_Packages_SMD:TO-263-7_TabPin4" H 5600 3550 60  0001 C CNN
 F 3 "" H 5600 3550 60  0001 C CNN
@@
 P 9750 3300
 F 0 "M6" H 9100 3600 60  0000 C CNN
-F 1 "IPB017N10N5" H 9100 3500 60  0000 C CNN
+F 1 "IPB044N15N5" H 9100 3500 60  0000 C CNN
 F 2 "TO_SOT_Packages_SMD:TO-263-7_TabPin4" H 9100 3500 60  0001 C CNN
 F 3 "" H 9100 3500 60  0001 C CNN
@@
 P 3750 2900
 F 0 "U1" H 3450 3325 50  0000 R CNN
-F 1 "AD8418" H 3450 3250 50  0000 R CNN
+F 1 "AD8205" H 3450 3250 50  0000 R CNN
 F 2 "Housings_SOIC:SO-8_5.3x6.2mm_Pitch1.27mm" H 3800 2550 50  0001 C CNN
 F 3 "" H 4400 2200 50  0001 C CNN
@@
 P 7200 3050
 F 0 "U2" H 6900 3475 50  0000 R CNN
-F 1 "AD8418" H 6900 3400 50  0000 R CNN
+F 1 "AD8205" H 6900 3400 50  0000 R CNN
 F 2 "Housings_SOIC:SO-8_5.3x6.2mm_Pitch1.27mm" H 7250 2700 50  0001 C CNN
 F 3 "" H 7850 2350 50  0001 C CNN
@@
 Wire Wire Line
 	9750 900  9750 1300
+Text HLabel 3250 2050 1    60   Output ~ 0
+PhaseADrain
+Wire Wire Line
+	3250 2050 3250 2400
+Connection ~ 3250 2400
+Text HLabel 6700 2250 1    60   Output ~ 0
+PhaseBDrain
+Wire Wire Line
+	6700 2250 6700 2550
+Connection ~ 6700 2550
 $EndSCHEMATC

Commit message: Converted to kicad 5
Parts:
- D1, D10, D2, D5, D6, D9: symbol D_Schottky -> Device:D_Schottky
- D11, D12, D3, D4, D7, D8: symbol D_Zener -> Device:D_Zener
- M1, M2, M3, M4, M5, M6: symbol IPB017N10N5 -> infineon:IPB017N10N5
- R1, R10, R11, R12, R13, R14, R2, R3, R4, R5, R6, R7, R8, R9: symbol R -> Device:R
- U1, U2: symbol AD8418 -> Amplifier_Current:AD8205
Connections:
- net labels added: PhaseASource, PhaseBSource
- net labels removed: PhaseADrain, PhaseBDrain
- wire segments 100 -> 154
