File: hardware/MOSFETS.sch (KiCad schematic (older format))
At the start: 34 parts, among them M1 IPB044N15N5, M2 IPB044N15N5, M3 IPB044N15N5, M4 IPB044N15N5, M5 IPB044N15N5, M6 IPB044N15N5, U1 AD8205, U2 AD8205

Commit message: updated routing and all plots
Parts:
- M1, M2, M3, M4, M5, M6: value IPB044N15N5 -> IPB017N10N5
Changed lines of the file:
@@
 P 2850 1800
 F 0 "M1" H 2200 2100 60  0000 C CNN
-F 1 "IPB044N15N5" H 2200 2000 60  0000 C CNN
+F 1 "IPB017N10N5" H 2200 2000 60  0000 C CNN
 F 2 "TO_SOT_Packages_SMD:TO-263-7_TabPin4" H 2200 2000 60  0001 C CNN
 F 3 "" H 2200 2000 60  0001 C CNN
@@
 P 6250 1800
 F 0 "M3" H 5600 2100 60  0000 C CNN
-F 1 "IPB044N15N5" H 5600 2000 60  0000 C CNN
+F 1 "IPB017N10N5" H 5600 2000 60  0000 C CNN
 F 2 "TO_SOT_Packages_SMD:TO-263-7_TabPin4" H 5600 2000 60  0001 C CNN
 F 3 "" H 5600 2000 60  0001 C CNN
@@
 P 9750 1750
 F 0 "M5" H 9100 2050 60  0000 C CNN
-F 1 "IPB044N15N5" H 9100 1950 60  0000 C CNN
+F 1 "IPB017N10N5" H 9100 1950 60  0000 C CNN
 F 2 "TO_SOT_Packages_SMD:TO-263-7_TabPin4" H 9100 1950 60  0001 C CNN
 F 3 "" H 9100 1950 60  0001 C CNN
@@
 P 2850 3350
 F 0 "M2" H 2200 3650 60  0000 C CNN
-F 1 "IPB044N15N5" H 2200 3550 60  0000 C CNN
+F 1 "IPB017N10N5" H 2200 3550 60  0000 C CNN
 F 2 "TO_SOT_Packages_SMD:TO-263-7_TabPin4" H 2200 3550 60  0001 C CNN
 F 3 "" H 2200 3550 60  0001 C CNN
@@
 P 6250 3350
 F 0 "M4" H 5600 3650 60  0000 C CNN
-F 1 "IPB044N15N5" H 5600 3550 60  0000 C CNN
+F 1 "IPB017N10N5" H 5600 3550 60  0000 C CNN
 F 2 "TO_SOT_Packages_SMD:TO-263-7_TabPin4" H 5600 3550 60  0001 C CNN
 F 3 "" H 5600 3550 60  0001 C CNN
@@
 P 9750 3300
 F 0 "M6" H 9100 3600 60  0000 C CNN
-F 1 "IPB044N15N5" H 9100 3500 60  0000 C CNN
+F 1 "IPB017N10N5" H 9100 3500 60  0000 C CNN
 F 2 "TO_SOT_Packages_SMD:TO-263-7_TabPin4" H 9100 3500 60  0001 C CNN
 F 3 "" H 9100 3500 60  0001 C CNN

Commit message: Updated schematic for additional capacitors
Parts:
- added C11, C12, C13, C14, C15, C16: 4.7u, symbol Device:CP1
Connections:
- wire segments 154 -> 183
Changed lines of the file:
@@
 	1800 900  2850 900
 Wire Wire Line
-	2850 900  2850 1350
-Wire Wire Line
-	6250 900  6250 1350
+	2850 900  2850 1150
+Wire Wire Line
+	6250 900  6250 1150
 Connection ~ 2850 900
 Text HLabel 1550 4800 0    60   UnSpc ~ 0
@@
 Connection ~ 2850 4800
 Connection ~ 6250 4800
-Wire Wire Line
-	9750 900  9750 1300
-Text HLabel 3250 2050 1    60   Output ~ 0
+Text HLabel 3450 2000 2    60   Output ~ 0
 PhaseASource
-Wire Wire Line
-	3250 2050 3250 2400
 Connection ~ 3250 2400
-Text HLabel 6700 2250 1    60   Output ~ 0
+Text HLabel 6900 2000 2    60   Output ~ 0
 PhaseBSource
-Wire Wire Line
-	6700 2250 6700 2550
 Connection ~ 6700 2550
 Wire Wire Line
@@
 Wire Wire Line
 	6700 2550 7000 2550
+Wire Wire Line
+	3250 2000 3450 2000
+Wire Wire Line
+	3250 2000 3250 2400
+Wire Wire Line
+	6700 2000 6900 2000
+Wire Wire Line
+	6700 2000 6700 2550
+$Comp
+L Device:CP1 C11
+U 1 1 5C53D027
+P 3400 1350
+F 0 "C11" H 3515 1441 50  0000 L CNN
+F 1 "4.7u" H 3515 1350 50  0000 L CNN
+F 2 "" H 3400 1350 50  0001 C CNN
+F 3 "~" H 3400 1350 50  0001 C CNN
+F 4 "UUR2A4R7MCL6GS" H 3200 1600 50  0000 L CNN "PN"
+	1    3400 1350
+	1    0    0    -1
+$EndComp
+Text Label 4250 1600 0    60   ~ 0
+GND
+Text Label 7500 1550 0    60   ~ 0
+GND
+Text Label 10650 1400 0    60   ~ 0
+GND
+Wire Wire Line
+	3400 1200 3400 1150
+Wire Wire Line
+	3400 1150 2850 1150
+Connection ~ 2850 1150
+Wire Wire Line
+	2850 1150 2850 1350
+Wire Wire Line
+	3850 1200 3850 1150
+Wire Wire Line
+	3850 1150 3400 1150
+Connection ~ 3400 1150
+Wire Wire Line
+	3400 1500 3400 1600
+Wire Wire Line
+	3400 1600 3850 1600
+Wire Wire Line
+	3850 1500 3850 1600
+Connection ~ 3850 1600
+Wire Wire Line
+	3850 1600 4250 1600
+Wire Wire Line
+	7100 1200 7100 1150
+Wire Wire Line
+	7100 1150 6700 1150
+Connection ~ 6250 1150
+Wire Wire Line
+	6250 1150 6250 1350
+Wire Wire Line
+	6700 1200 6700 1150
+Connection ~ 6700 1150
+Wire Wire Line
+	6700 1150 6250 1150
+Wire Wire Line
+	6700 1500 6700 1550
+Wire Wire Line
+	6700 1550 7100 1550
+Wire Wire Line
+	7100 1500 7100 1550
+Connection ~ 7100 1550
+Wire Wire Line
+	7100 1550 7500 1550
+Wire Wire Line
+	10050 1000 10050 950
+Wire Wire Line
+	10450 1000 10450 950
+Wire Wire Line
+	10450 950  10050 950
+Wire Wire Line
+	10050 1300 10050 1400
+Wire Wire Line
+	10050 1400 10450 1400
+Wire Wire Line
+	10450 1300 10450 1400
+Connection ~ 10450 1400
+Wire Wire Line
+	10450 1400 10650 1400
+$Comp
+L Device:CP1 C12
+U 1 1 5C59D030
+P 3850 1350
+F 0 "C12" H 3965 1441 50  0000 L CNN
+F 1 "4.7u" H 3965 1350 50  0000 L CNN
+F 2 "" H 3850 1350 50  0001 C CNN
+F 3 "~" H 3850 1350 50  0001 C CNN
+F 4 "UUR2A4R7MCL6GS" H 4000 1250 50  0000 L CNN "PN"
+	1    3850 1350
+	1    0    0    -1
+$EndComp
+$Comp
+L Device:CP1 C13
+U 1 1 5C59D09C
+P 6700 1350
+F 0 "C13" H 6815 1441 50  0000 L CNN
+F 1 "4.7u" H 6815 1350 50  0000 L CNN
+F 2 "" H 6700 1350 50  0001 C CNN
+F 3 "~" H 6700 1350 50  0001 C CNN
+F 4 "UUR2A4R7MCL6GS" H 6500 1600 50  0000 L CNN "PN"
+	1    6700 1350
+	1    0    0    -1
+$EndComp
+$Comp
+L Device:CP1 C14
+U 1 1 5C59D13E
+P 7100 1350
+F 0 "C14" H 7200 1500 50  0000 L CNN
+F 1 "4.7u" H 7200 1400 50  0000 L CNN
+F 2 "" H 7100 1350 50  0001 C CNN
+F 3 "~" H 7100 1350 50  0001 C CNN
+F 4 "UUR2A4R7MCL6GS" H 7250 1300 50  0000 L CNN "PN"
+	1    7100 1350
+	1    0    0    -1
+$EndComp
+$Comp
+L Device:CP1 C15
+U 1 1 5C59D1AC
+P 10050 1150
+F 0 "C15" H 10165 1241 50  0000 L CNN
+F 1 "4.7u" H 10165 1150 50  0000 L CNN
+F 2 "" H 10050 1150 50  0001 C CNN
+F 3 "~" H 10050 1150 50  0001 C CNN
+F 4 "UUR2A4R7MCL6GS" H 9800 1400 50  0000 L CNN "PN"
+	1    10050 1150
+	1    0    0    -1
+$EndComp
+$Comp
+L Device:CP1 C16
+U 1 1 5C59D44A
+P 10450 1150
+F 0 "C16" H 10565 1241 50  0000 L CNN
+F 1 "4.7u" H 10565 1150 50  0000 L CNN
+F 2 "" H 10450 1150 50  0001 C CNN
+F 3 "~" H 10450 1150 50  0001 C CNN
+F 4 "UUR2A4R7MCL6GS" H 10500 1050 50  0000 L CNN "PN"
+	1    10450 1150
+	1    0    0    -1
+$EndComp
+Wire Wire Line
+	9750 900  9750 950
+Wire Wire Line
+	10050 950  9750 950
+Connection ~ 10050 950
+Connection ~ 9750 950
+Wire Wire Line
+	9750 950  9750 1300
 $EndSCHEMATC

Commit message: Added additional capacitors for 48v bus
Parts:
- C11, C12, C13, C14, C15, C16: footprint (none) -> Capacitors_SMD:CP_Elec_8x6.5
Changed lines of the file:
@@
 F 0 "C11" H 3515 1441 50  0000 L CNN
 F 1 "4.7u" H 3515 1350 50  0000 L CNN
-F 2 "" H 3400 1350 50  0001 C CNN
+F 2 "Capacitors_SMD:CP_Elec_8x6.5" H 3400 1350 50  0001 C CNN
 F 3 "~" H 3400 1350 50  0001 C CNN
 F 4 "UUR2A4R7MCL6GS" H 3200 1600 50  0000 L CNN "PN"
@@
 F 0 "C12" H 3965 1441 50  0000 L CNN
 F 1 "4.7u" H 3965 1350 50  0000 L CNN
-F 2 "" H 3850 1350 50  0001 C CNN
+F 2 "Capacitors_SMD:CP_Elec_8x6.5" H 3850 1350 50  0001 C CNN
 F 3 "~" H 3850 1350 50  0001 C CNN
 F 4 "UUR2A4R7MCL6GS" H 4000 1250 50  0000 L CNN "PN"
@@
 F 0 "C13" H 6815 1441 50  0000 L CNN
 F 1 "4.7u" H 6815 1350 50  0000 L CNN
-F 2 "" H 6700 1350 50  0001 C CNN
+F 2 "Capacitors_SMD:CP_Elec_8x6.5" H 6700 1350 50  0001 C CNN
 F 3 "~" H 6700 1350 50  0001 C CNN
 F 4 "UUR2A4R7MCL6GS" H 6500 1600 50  0000 L CNN "PN"
@@
 F 0 "C14" H 7200 1500 50  0000 L CNN
 F 1 "4.7u" H 7200 1400 50  0000 L CNN
-F 2 "" H 7100 1350 50  0001 C CNN
+F 2 "Capacitors_SMD:CP_Elec_8x6.5" H 7100 1350 50  0001 C CNN
 F 3 "~" H 7100 1350 50  0001 C CNN
 F 4 "UUR2A4R7MCL6GS" H 7250 1300 50  0000 L CNN "PN"
@@
 F 0 "C15" H 10165 1241 50  0000 L CNN
 F 1 "4.7u" H 10165 1150 50  0000 L CNN
-F 2 "" H 10050 1150 50  0001 C CNN
+F 2 "Capacitors_SMD:CP_Elec_8x6.5" H 10050 1150 50  0001 C CNN
 F 3 "~" H 10050 1150 50  0001 C CNN
 F 4 "UUR2A4R7MCL6GS" H 9800 1400 50  0000 L CNN "PN"
@@
 F 0 "C16" H 10565 1241 50  0000 L CNN
 F 1 "4.7u" H 10565 1150 50  0000 L CNN
-F 2 "" H 10450 1150 50  0001 C CNN
+F 2 "Capacitors_SMD:CP_Elec_8x6.5" H 10450 1150 50  0001 C CNN
 F 3 "~" H 10450 1150 50  0001 C CNN
 F 4 "UUR2A4R7MCL6GS" H 10500 1050 50  0000 L CNN "PN"
