File: hardware/Microcontroller.sch (KiCad schematic (older format))
At the start: 1 part

Commit message: cleaned up schematic
Other:
- note added: "STM uses five 2x5 0.1" female headers on each side\nPN: M20-7810545"

Commit message: annotated schematic
Parts:
- gave numbers to parts that had none: 1
Changed lines of the file:
@@
 $EndDescr
 $Comp
-L STM32F4-DISCOVERY M?
+L STM32F4-DISCOVERY M1
 U 1 1 5AB69504
 P 3750 2200
-F 0 "M?" H 3750 2200 45  0001 C CNN
+F 0 "M1" H 3750 2200 45  0001 C CNN
 F 1 "STM32F4-DISCOVERY" H 3750 2200 45  0001 C CNN
 F 2 "STM32F4-DISCOVERY-SIMON_STM32F4-DISCOVERY" H 3780 2350 20  0001 C CNN

Commit message: created new footprints, modified schematic
Parts:
- M7: renamed from M1; footprint STM32F4-DISCOVERY-SIMON_STM32F4-DISCOVERY -> custom:STM32-F4-DISCOVERY
Connections:
- net labels added: I2C_SCL, I2C_SDA
- net labels removed: Throttle
- wire segments 28 -> 29
- no-connect marks 0 -> 73
Other:
- note added: "STM uses five 2x25 0.1" female headers on each side\nPN: NPPC252KFMS-RC"
- note removed: "STM uses five 2x5 0.1" female headers on each side\nPN: M20-7810545"
