File: hardware/Microcontroller.sch (KiCad schematic (older format))
At the start: 1 part, among them M7 STM32F4-DISCOVERY

Commit message: Converted to kicad 5
Parts:
- M7: symbol STM32F4-DISCOVERY -> STM32F4-DISCOVERY-SIMON:STM32F4-DISCOVERY
Changed lines of the file:
@@
-EESchema Schematic File Version 2
-LIBS:power
-LIBS:device
-LIBS:switches
-LIBS:relays
-LIBS:motors
-LIBS:transistors
-LIBS:conn
-LIBS:linear
-LIBS:regul
-LIBS:74xx
-LIBS:cmos4000
-LIBS:adc-dac
-LIBS:memory
-LIBS:xilinx
-LIBS:microcontrollers
-LIBS:dsp
-LIBS:microchip
-LIBS:analog_switches
-LIBS:motorola
-LIBS:texas
-LIBS:intel
-LIBS:audio
-LIBS:interface
-LIBS:digital-audio
-LIBS:philips
-LIBS:display
-LIBS:cypress
-LIBS:siliconi
-LIBS:opto
-LIBS:atmel
-LIBS:contrib
-LIBS:valves
-LIBS:infineon
-LIBS:crf_1
-LIBS:STM32F4-DISCOVERY-SIMON
-LIBS:bldc_v1-cache
-EELAYER 25 0
+EESchema Schematic File Version 4
+EELAYER 26 0
 EELAYER END
 $Descr A4 11693 8268
@@
 $EndDescr
 $Comp
-L STM32F4-DISCOVERY M7
+L STM32F4-DISCOVERY-SIMON:STM32F4-DISCOVERY M7
 U 1 1 5AB69504
 P 3750 2200
