File: hardware/PowerConverter.sch (KiCad schematic (older format))
At the start: 13 parts

Commit message: annotated schematic
Parts:
- renumbered 12vConverter to 12vConverter1, 5vConverter to 5vConverter1, C3 to C7, C4 to C8, C1 to C9, D1 to D13, D2 to D14, R2 to R16, R1 to R17, R4 to R18, R3 to R19
Changed lines of the file:
@@
 $EndDescr
 $Comp
-L TL2575HV 12vConverter
+L TL2575HV 12vConverter1
 U 1 1 5AB4721C
 P 3200 1450
-F 0 "12vConverter" H 3200 1950 60  0000 C CNN
+F 0 "12vConverter1" H 3200 1950 60  0000 C CNN
 F 1 "TL2575HV" H 3200 1850 60  0000 C CNN
 F 2 "" H 3150 1450 60  0001 C CNN
@@
 $EndComp
 $Comp
-L TL2575HV 5vConverter
+L TL2575HV 5vConverter1
 U 1 1 5AB4724C
 P 3200 3900
-F 0 "5vConverter" H 3200 4400 60  0000 C CNN
+F 0 "5vConverter1" H 3200 4400 60  0000 C CNN
 F 1 "TL2575HV" H 3200 4300 60  0000 C CNN
 F 2 "" H 3150 3900 60  0001 C CNN
@@
 $EndComp
 $Comp
-L R R1
+L R R17
 U 1 1 5AB473CB
 P 5200 2200
-F 0 "R1" V 5280 2200 50  0000 C CNN
+F 0 "R17" V 5280 2200 50  0000 C CNN
 F 1 "2k" V 5200 2200 50  0000 C CNN
 F 2 "" V 5130 2200 50  0001 C CNN
@@
 $EndComp
 $Comp
-L R R2
+L R R16
 U 1 1 5AB47408
 P 5200 1700
-F 0 "R2" V 5280 1700 50  0000 C CNN
+F 0 "R16" V 5280 1700 50  0000 C CNN
 F 1 "18k" V 5200 1700 50  0000 C CNN
 F 2 "" V 5130 1700 50  0001 C CNN
@@
 $EndComp
 $Comp
-L R R4
+L R R18
 U 1 1 5AB4745C
 P 5300 4100
-F 0 "R4" V 5380 4100 50  0000 C CNN
+F 0 "R18" V 5380 4100 50  0000 C CNN
 F 1 "6.04k" V 5300 4100 50  0000 C CNN
 F 2 "" V 5230 4100 50  0001 C CNN
@@
 $EndComp
 $Comp
-L R R3
+L R R19
 U 1 1 5AB47CAF
 P 5300 4600
-F 0 "R3" V 5380 4600 50  0000 C CNN
+F 0 "R19" V 5380 4600 50  0000 C CNN
 F 1 "2k" V 5300 4600 50  0000 C CNN
 F 2 "" V 5230 4600 50  0001 C CNN
@@
 	3900 1450 3750 1450
 $Comp
-L C C1
+L C C9
 U 1 1 5AB48931
 P 4500 1900
-F 0 "C1" H 4525 2000 50  0000 L CNN
+F 0 "C9" H 4525 2000 50  0000 L CNN
 F 1 "330uF" H 4525 1800 50  0000 L CNN
 F 2 "" H 4538 1750 50  0001 C CNN
@@
 Connection ~ 4500 2450
 $Comp
-L D_Schottky D1
+L D_Schottky D13
 U 1 1 5AB48BB4
 P 3800 1950
-F 0 "D1" H 3800 2050 50  0000 C CNN
+F 0 "D13" H 3800 2050 50  0000 C CNN
 F 1 "NRVTS260ESFT1G" H 3800 1850 50  0000 C CNN
 F 2 "" H 3800 1950 50  0001 C CNN
@@
 Connection ~ 3000 4850
 $Comp
-L D_Schottky D2
+L D_Schottky D14
 U 1 1 5AB4996E
 P 3800 4350
-F 0 "D2" H 3800 4450 50  0000 C CNN
+F 0 "D14" H 3800 4450 50  0000 C CNN
 F 1 "NRVTS260ESFT1G" H 3800 4250 50  0000 C CNN
 F 2 "" H 3800 4350 50  0001 C CNN
@@
 Connection ~ 3800 1450
 $Comp
-L C C3
+L C C7
 U 1 1 5AB49CE1
 P 2400 1700
-F 0 "C3" H 2425 1800 50  0000 L CNN
+F 0 "C7" H 2425 1800 50  0000 L CNN
 F 1 "100uF" H 2425 1600 50  0000 L CNN
 F 2 "" H 2438 1550 50  0001 C CNN
@@
 Connection ~ 2400 2450
 $Comp
-L C C4
+L C C8
 U 1 1 5AB49F15
 P 2400 4150
-F 0 "C4" H 2425 4250 50  0000 L CNN
+F 0 "C8" H 2425 4250 50  0000 L CNN
 F 1 "100uF" H 2425 4050 50  0000 L CNN
 F 2 "" H 2438 4000 50  0001 C CNN

Commit message: created new footprints, modified schematic
Parts:
- removed C9: 330uF, symbol C
- added C10: 1200uF, Capacitors_SMD:CP_Elec_10x10, symbol CP
- added C9: 330uF, Capacitors_SMD:CP_Elec_8x10, symbol CP
- 12vConverter1, 5vConverter1: footprint (none) -> TO_SOT_Packages_SMD:TO-263-5_TabPin3
- C7, C8: footprint (none) -> Capacitors_SMD:CP_Elec_10x10
- D13, D14: footprint (none) -> Diodes_SMD:D_SOD-123F
- L1: footprint (none) -> Inductors_THT:L_Toroid_Horizontal_D32.5mm_P30.00mm_Bourns_2300; PN 60B684C -> 2322-H-RC
- L2: footprint (none) -> Inductors_THT:L_Toroid_Horizontal_D24.1mm_P23.10mm_Bourns_2200; PN 33331C -> 2200HT-331-H-RC
- R15: renamed from R16; footprint (none) -> Resistors_SMD:R_0805_HandSoldering
- R16: renamed from R17; footprint (none) -> Resistors_SMD:R_0603_HandSoldering
- R17: renamed from R18; footprint (none) -> Resistors_SMD:R_0603_HandSoldering
- R18: renamed from R19; footprint (none) -> Resistors_SMD:R_0603_HandSoldering
Connections:
- wire segments 36 -> 38
Changed lines of the file:
@@
 F 0 "12vConverter1" H 3200 1950 60  0000 C CNN
 F 1 "TL2575HV" H 3200 1850 60  0000 C CNN
-F 2 "" H 3150 1450 60  0001 C CNN
+F 2 "TO_SOT_Packages_SMD:TO-263-5_TabPin3" H 3150 1450 60  0001 C CNN
 F 3 "" H 3150 1450 60  0001 C CNN
 	1    3200 1450
@@
 F 0 "5vConverter1" H 3200 4400 60  0000 C CNN
 F 1 "TL2575HV" H 3200 4300 60  0000 C CNN
-F 2 "" H 3150 3900 60  0001 C CNN
+F 2 "TO_SOT_Packages_SMD:TO-263-5_TabPin3" H 3150 3900 60  0001 C CNN
 F 3 "" H 3150 3900 60  0001 C CNN
 	1    3200 3900
@@
 $EndComp
 $Comp
-L R R17
+L R R16
 U 1 1 5AB473CB
 P 5200 2200
-F 0 "R17" V 5280 2200 50  0000 C CNN
+F 0 "R16" V 5280 2200 50  0000 C CNN
 F 1 "2k" V 5200 2200 50  0000 C CNN
-F 2 "" V 5130 2200 50  0001 C CNN
+F 2 "Resistors_SMD:R_0603_HandSoldering" V 5130 2200 50  0001 C CNN
 F 3 "" H 5200 2200 50  0001 C CNN
 F 4 "RR0816P-202-D " H 5750 2200 60  0000 C CNN "PN"
@@
 $EndComp
 $Comp
-L R R16
+L R R15
 U 1 1 5AB47408
 P 5200 1700
-F 0 "R16" V 5280 1700 50  0000 C CNN
+F 0 "R15" V 5280 1700 50  0000 C CNN
 F 1 "18k" V 5200 1700 50  0000 C CNN
-F 2 "" V 5130 1700 50  0001 C CNN
+F 2 "Resistors_SMD:R_0805_HandSoldering" V 5130 1700 50  0001 C CNN
 F 3 "" H 5200 1700 50  0001 C CNN
 F 4 "ERA-6AEB183V" H 5650 1700 60  0000 C CNN "PN"
@@
 $EndComp
 $Comp
-L R R18
+L R R17
 U 1 1 5AB4745C
 P 5300 4100
-F 0 "R18" V 5380 4100 50  0000 C CNN
+F 0 "R17" V 5380 4100 50  0000 C CNN
 F 1 "6.04k" V 5300 4100 50  0000 C CNN
-F 2 "" V 5230 4100 50  0001 C CNN
+F 2 "Resistors_SMD:R_0603_HandSoldering" V 5230 4100 50  0001 C CNN
 F 3 "" H 5300 4100 50  0001 C CNN
 F 4 "ERA-3AEB6041V" H 5850 4100 60  0000 C CNN "PN"
@@
 $EndComp
 $Comp
-L R R19
+L R R18
 U 1 1 5AB47CAF
 P 5300 4600
-F 0 "R19" V 5380 4600 50  0000 C CNN
+F 0 "R18" V 5380 4600 50  0000 C CNN
 F 1 "2k" V 5300 4600 50  0000 C CNN
-F 2 "" V 5230 4600 50  0001 C CNN
+F 2 "Resistors_SMD:R_0603_HandSoldering" V 5230 4600 50  0001 C CNN
 F 3 "" H 5300 4600 50  0001 C CNN
 F 4 "RR0816P-202-D " H 5850 4600 60  0000 C CNN "PN"
@@
 F 0 "L1" V 4000 1450 50  0000 C CNN
 F 1 "680uH" V 4125 1450 50  0000 C CNN
-F 2 "" H 4050 1450 50  0001 C CNN
+F 2 "Inductors_THT:L_Toroid_Horizontal_D32.5mm_P30.00mm_Bourns_2300" H 4050 1450 50  0001 C CNN
 F 3 "" H 4050 1450 50  0001 C CNN
-F 4 "60B684C" V 3900 1450 60  0000 C CNN "PN"
+F 4 "2322-H-RC" V 3900 1400 60  0000 C CNN "PN"
 	1    4050 1450
 	0    -1   -1   0
@@
 48v
 Wire Wire Line
-	3900 1450 3750 1450
-$Comp
-L C C9
-U 1 1 5AB48931
-P 4500 1900
-F 0 "C9" H 4525 2000 50  0000 L CNN
-F 1 "330uF" H 4525 1800 50  0000 L CNN
-F 2 "" H 4538 1750 50  0001 C CNN
-F 3 "" H 4500 1900 50  0001 C CNN
-F 4 "EEE-1EA331UP" V 4350 1800 60  0000 C CNN "PN"
-	1    4500 1900
-	1    0    0    -1
-$EndComp
+	3750 1450 3900 1450
 Wire Wire Line
 	4500 1750 4500 1450
@@
 F 0 "D13" H 3800 2050 50  0000 C CNN
 F 1 "NRVTS260ESFT1G" H 3800 1850 50  0000 C CNN
-F 2 "" H 3800 1950 50  0001 C CNN
+F 2 "Diodes_SMD:D_SOD-123F" H 3800 1950 50  0001 C CNN
 F 3 "" H 3800 1950 50  0001 C CNN
 	1    3800 1950
@@
 F 0 "L2" V 4100 3900 50  0000 C CNN
 F 1 "330uH" V 4225 3900 50  0000 C CNN
-F 2 "" H 4150 3900 50  0001 C CNN
+F 2 "Inductors_THT:L_Toroid_Horizontal_D24.1mm_P23.10mm_Bourns_2200" H 4150 3900 50  0001 C CNN
 F 3 "" H 4150 3900 50  0001 C CNN
-F 4 "33331C" V 4000 3900 60  0000 C CNN "PN"
+F 4 "2200HT-331-H-RC" V 4000 3800 60  0000 C CNN "PN"
 	1    4150 3900
 	0    -1   -1   0
 $EndComp
 Wire Wire Line
-	4000 3900 3750 3900
+	3750 3900 4000 3900
 Wire Wire Line
 	4300 3900 5750 3900
@@
 	5300 3900 5300 3950
 Wire Wire Line
-	5300 4450 5300 4250
+	5300 4250 5300 4450
 Wire Wire Line
 	5300 4350 5050 4350
@@
 Wire Wire Line
 	2100 3650 2600 3650
-Text Label 2100 4850 2    60   ~ 0
-GND
-Wire Wire Line
-	2100 4850 5300 4850
-Wire Wire Line
-	5300 4850 5300 4750
-Wire Wire Line
-	3350 4450 3350 4850
-Connection ~ 3350 4850
-Wire Wire Line
-	3000 4450 3000 4850
-Connection ~ 3000 4850
+Text Label 2100 4900 2    60   ~ 0
+GND
+Wire Wire Line
+	2100 4900 5300 4900
+Wire Wire Line
+	5300 4900 5300 4750
+Wire Wire Line
+	3350 4450 3350 4900
+Connection ~ 3350 4900
+Wire Wire Line
+	3000 4450 3000 4900
+Connection ~ 3000 4900
 $Comp
 L D_Schottky D14
@@
 F 0 "D14" H 3800 4450 50  0000 C CNN
 F 1 "NRVTS260ESFT1G" H 3800 4250 50  0000 C CNN
-F 2 "" H 3800 4350 50  0001 C CNN
+F 2 "Diodes_SMD:D_SOD-123F" H 3800 4350 50  0001 C CNN
 F 3 "" H 3800 4350 50  0001 C CNN
 	1    3800 4350
@@
 Connection ~ 3800 3900
 Wire Wire Line
-	3800 4500 3800 4850
-Connection ~ 3800 4850
+	3800 4500 3800 4900
+Connection ~ 3800 4900
 Wire Wire Line
 	3800 2100 3800 2450
@@
 F 0 "C7" H 2425 1800 50  0000 L CNN
 F 1 "100uF" H 2425 1600 50  0000 L CNN
-F 2 "" H 2438 1550 50  0001 C CNN
+F 2 "Capacitors_SMD:CP_Elec_10x10" H 2438 1550 50  0001 C CNN
 F 3 "" H 2400 1700 50  0001 C CNN
 F 4 " EEE-1JA101P" V 2250 1600 60  0000 C CNN "PN"
@@
 F 0 "C8" H 2425 4250 50  0000 L CNN
 F 1 "100uF" H 2425 4050 50  0000 L CNN
-F 2 "" H 2438 4000 50  0001 C CNN
+F 2 "Capacitors_SMD:CP_Elec_10x10" H 2438 4000 50  0001 C CNN
 F 3 "" H 2400 4150 50  0001 C CNN
 F 4 " EEE-1JA101P" V 2250 4050 60  0000 C CNN "PN"
@@
 Connection ~ 2400 3650
 Wire Wire Line
-	2400 4300 2400 4850
-Connection ~ 2400 4850
+	2400 4300 2400 4900
+Connection ~ 2400 4900
+$Comp
+L CP C10
+U 1 1 5ABA051A
+P 4800 4300
+F 0 "C10" H 4825 4400 50  0000 L CNN
+F 1 "1200uF" H 4825 4200 50  0000 L CNN
+F 2 "Capacitors_SMD:CP_Elec_10x10" H 4838 4150 50  0001 C CNN
+F 3 "" H 4800 4300 50  0001 C CNN
+F 4 "UCL1A122MNL1GS" V 4650 4100 60  0000 C CNN "PN"
+	1    4800 4300
+	1    0    0    -1
+$EndComp
+$Comp
+L CP C9
+U 1 1 5ABA0583
+P 4500 1900
+F 0 "C9" H 4525 2000 50  0000 L CNN
+F 1 "330uF" H 4525 1800 50  0000 L CNN
+F 2 "Capacitors_SMD:CP_Elec_8x10" H 4538 1750 50  0001 C CNN
+F 3 "" H 4500 1900 50  0001 C CNN
+F 4 "EEE-1EA331UP" V 4350 1800 60  0000 C CNN "PN"
+	1    4500 1900
+	1    0    0    -1
+$EndComp
+Wire Wire Line
+	4800 4150 4800 3900
+Connection ~ 4800 3900
+Wire Wire Line
+	4800 4450 4800 4900
+Connection ~ 4800 4900
 $EndSCHEMATC
