File: hardware/PowerConverter.sch (KiCad schematic (older format))
At the start: 14 parts

Commit message: Converted to kicad 5
Parts:
- 12vConverter1, 5vConverter1: symbol TL2575HV -> infineon:TL2575HV
- C10, C9: symbol CP -> Device:CP
- C7, C8: symbol C -> Device:C
- D13, D14: symbol D_Schottky -> Device:D_Schottky
- L1, L2: symbol L -> Device:L
- R15, R16, R17, R18: symbol R -> Device:R
Changed lines of the file:
@@
-EESchema Schematic File Version 2
-LIBS:power
-LIBS:device
-LIBS:switches
-LIBS:relays
-LIBS:motors
-LIBS:transistors
-LIBS:conn
-LIBS:linear
-LIBS:regul
-LIBS:74xx
-LIBS:cmos4000
-LIBS:adc-dac
-LIBS:memory
-LIBS:xilinx
-LIBS:microcontrollers
-LIBS:dsp
-LIBS:microchip
-LIBS:analog_switches
-LIBS:motorola
-LIBS:texas
-LIBS:intel
-LIBS:audio
-LIBS:interface
-LIBS:digital-audio
-LIBS:philips
-LIBS:display
-LIBS:cypress
-LIBS:siliconi
-LIBS:opto
-LIBS:atmel
-LIBS:contrib
-LIBS:valves
-LIBS:infineon
-LIBS:crf_1
-LIBS:STM32F4-DISCOVERY-SIMON
-LIBS:bldc_v1-cache
-EELAYER 25 0
+EESchema Schematic File Version 4
+EELAYER 26 0
 EELAYER END
 $Descr A4 11693 8268
@@
 $EndDescr
 $Comp
-L TL2575HV 12vConverter1
+L infineon:TL2575HV 12vConverter1
 U 1 1 5AB4721C
 P 3200 1450
@@
 $EndComp
 $Comp
-L TL2575HV 5vConverter1
+L infineon:TL2575HV 5vConverter1
 U 1 1 5AB4724C
 P 3200 3900
@@
 $EndComp
 $Comp
-L R R16
+L Device:R R16
 U 1 1 5AB473CB
 P 5200 2200
@@
 $EndComp
 $Comp
-L R R15
+L Device:R R15
 U 1 1 5AB47408
 P 5200 1700
@@
 $EndComp
 $Comp
-L R R17
+L Device:R R17
 U 1 1 5AB4745C
 P 5300 4100
@@
 $EndComp
 $Comp
-L R R18
+L Device:R R18
 U 1 1 5AB47CAF
 P 5300 4600
@@
 $EndComp
 $Comp
-L L L1
+L Device:L L1
 U 1 1 5AB48433
 P 4050 1450
@@
 Connection ~ 4500 2450
 $Comp
-L D_Schottky D13
+L Device:D_Schottky D13
 U 1 1 5AB48BB4
 P 3800 1950
@@
 	2150 1200 2600 1200
 $Comp
-L L L2
+L Device:L L2
 U 1 1 5AB492B5
 P 4150 3900
@@
 Connection ~ 3000 4900
 $Comp
-L D_Schottky D14
+L Device:D_Schottky D14
 U 1 1 5AB4996E
 P 3800 4350
@@
 Connection ~ 3800 1450
 $Comp
-L C C7
+L Device:C C7
 U 1 1 5AB49CE1
 P 2400 1700
@@
 Connection ~ 2400 2450
 $Comp
-L C C8
+L Device:C C8
 U 1 1 5AB49F15
 P 2400 4150
@@
 Connection ~ 2400 4900
 $Comp
-L CP C10
+L Device:CP C10
 U 1 1 5ABA051A
 P 4800 4300
@@
 $EndComp
 $Comp
-L CP C9
+L Device:CP C9
 U 1 1 5ABA0583
 P 4500 1900
