File: hardware/PowerConverter.sch (KiCad schematic (older format))
At the start: 14 parts

Commit message: Updated schematic for additional capacitors
Connections:
- wire segments 38 -> 58
Changed lines of the file:
@@
 $EndComp
 Wire Wire Line
-	4200 1450 5600 1450
+	4200 1450 4500 1450
 Wire Wire Line
 	5200 1450 5200 1550
 Wire Wire Line
-	5200 1850 5200 2050
+	5200 1850 5200 1950
 Wire Wire Line
 	3750 1200 5000 1200
@@
 	5200 2450 5200 2350
 Wire Wire Line
-	2150 2450 5200 2450
+	2150 2450 2400 2450
 Wire Wire Line
 	3350 2450 3350 2000
@@
 48v
 Wire Wire Line
-	3750 1450 3900 1450
+	3750 1450 3800 1450
 Wire Wire Line
 	4500 1750 4500 1450
@@
 $EndComp
 Wire Wire Line
-	2150 1200 2600 1200
+	2150 1200 2400 1200
 $Comp
 L Device:L L2
@@
 $EndComp
 Wire Wire Line
-	3750 3900 4000 3900
-Wire Wire Line
-	4300 3900 5750 3900
+	3750 3900 3800 3900
+Wire Wire Line
+	4300 3900 4800 3900
 Wire Wire Line
 	5300 3900 5300 3950
 Wire Wire Line
-	5300 4250 5300 4450
+	5300 4250 5300 4350
 Wire Wire Line
 	5300 4350 5050 4350
@@
 48v
 Wire Wire Line
-	2100 3650 2600 3650
+	2100 3650 2400 3650
 Text Label 2100 4900 2    60   ~ 0
 GND
 Wire Wire Line
-	2100 4900 5300 4900
+	2100 4900 2400 4900
 Wire Wire Line
 	5300 4900 5300 4750
@@
 	4800 4450 4800 4900
 Connection ~ 4800 4900
+Wire Wire Line
+	5200 1950 5200 2050
+Wire Wire Line
+	3350 2450 3800 2450
+Wire Wire Line
+	3000 2450 3350 2450
+Wire Wire Line
+	5200 1450 5600 1450
+Wire Wire Line
+	4500 1450 5200 1450
+Wire Wire Line
+	4500 2450 5200 2450
+Wire Wire Line
+	5300 4350 5300 4450
+Wire Wire Line
+	5300 3900 5750 3900
+Wire Wire Line
+	3350 4900 3800 4900
+Wire Wire Line
+	3000 4900 3350 4900
+Wire Wire Line
+	3800 3900 4000 3900
+Wire Wire Line
+	3800 4900 4800 4900
+Wire Wire Line
+	3800 2450 4500 2450
+Wire Wire Line
+	3800 1450 3900 1450
+Wire Wire Line
+	2400 1200 2600 1200
+Wire Wire Line
+	2400 2450 3000 2450
+Wire Wire Line
+	2400 3650 2600 3650
+Wire Wire Line
+	2400 4900 3000 4900
+Wire Wire Line
+	4800 3900 5300 3900
+Wire Wire Line
+	4800 4900 5300 4900
 $EndSCHEMATC

Commit message: Added additional capacitors for 48v bus
Parts:
- C10: symbol Device:CP -> Device:CP1
- C7, C8: symbol Device:C -> Device:CP1
- C9: footprint Capacitors_SMD:CP_Elec_8x10 -> Capacitors_SMD:CP_Elec_8x10.5; symbol Device:CP -> Device:CP1
Changed lines of the file:
@@
 Connection ~ 3800 1450
 $Comp
-L Device:C C7
+L Device:CP1 C7
 U 1 1 5AB49CE1
 P 2400 1700
@@
 Connection ~ 2400 2450
 $Comp
-L Device:C C8
+L Device:CP1 C8
 U 1 1 5AB49F15
 P 2400 4150
@@
 Connection ~ 2400 4900
 $Comp
-L Device:CP C10
+L Device:CP1 C10
 U 1 1 5ABA051A
 P 4800 4300
@@
 $EndComp
 $Comp
-L Device:CP C9
+L Device:CP1 C9
 U 1 1 5ABA0583
 P 4500 1900
 F 0 "C9" H 4525 2000 50  0000 L CNN
 F 1 "330uF" H 4525 1800 50  0000 L CNN
-F 2 "Capacitors_SMD:CP_Elec_8x10" H 4538 1750 50  0001 C CNN
+F 2 "Capacitors_SMD:CP_Elec_8x10.5" H 4538 1750 50  0001 C CNN
 F 3 "" H 4500 1900 50  0001 C CNN
 F 4 "EEE-1EA331UP" V 4350 1800 60  0000 C CNN "PN"
