File: hardware/bldc_v1.kicad_pcb (KiCad board)
At the start: 2 copper layers, 63 parts, among them J1 Conn_01x06, J2 1x2_ScrewTerminal_65A, J3 Screw_Terminal_01x05, J4 RJ45, J5 Screw_Terminal_01x03, M1 IPB017N10N5, M2 IPB017N10N5, M3 IPB017N10N5, M4 IPB017N10N5, M5 IPB017N10N5, M6 IPB017N10N5, M7 STM32F4-DISCOVERY, U1 AD8418, U2 AD8418

Commit message: layed parts out on board
Parts:
- C1, C2, C3: footprint Capacitors_SMD:C_0402 -> Capacitors_SMD:C_0805_HandSoldering; moved to B.Cu
- C4, C5, C6, D10, M2, M4, M6, M7, R10, U1, U2: moved to B.Cu
- moved D13 188.9 mm to (91.6, 68.1), turned to 90 degrees
- moved R5 162.2 mm to (190.1, 69.6)
- moved J2 150.7 mm to (166.4, 41.8)
- moved R17 148.3 mm to (116.3, 64.4), turned to 180 degrees
- moved R15 141.3 mm to (96.3, 72.0)
- moved R1 138.6 mm to (157.7, 72.6), turned to 180 degrees
- moved D9 132.3 mm to (159.8, 118.1)
- moved D1 130.1 mm to (157.5, 68.1)
- moved R8 129.3 mm to (162.4, 104.6), turned to 90 degrees
- moved R4 124.9 mm to (162.6, 87.9), turned to 90 degrees
- moved R7 124.5 mm to (148.1, 103.9), turned to 180 degrees
- moved R2 123.4 mm to (147.8, 79.8), turned to 180 degrees
- moved C7 118.6 mm to (190.5, 48.4), turned to 90 degrees
- moved L1 118.0 mm to (93.0, 78.2), turned to 270 degrees
- moved U1 117.5 mm to (146.8, 65.5), turned to 180 degrees
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Connections:
- J5 pad 1: /GateDriver/PhaseC -> /GateDriver/PhaseA
- J5 pad 3: /GateDriver/PhaseA -> /GateDriver/PhaseC
- PhaseA1 pad 9: (no net) -> /GND
- PhaseB1 pad 9: (no net) -> /GND
- PhaseC1 pad 9: (no net) -> /GND
Other:
- board outline added: 135.4 x 108.3 mm

Commit message: finished board layout
Parts:
- added REF**: MountingHole_6.4mm_M6, Mounting_Holes:MountingHole_6.4mm_M6, F.Cu at (237.4, 48.9)
- added REF**: MountingHole_6.4mm_M6, Mounting_Holes:MountingHole_6.4mm_M6, F.Cu at (237.1, 130.0)
- added REF**: MountingHole_6.4mm_M6, Mounting_Holes:MountingHole_6.4mm_M6, F.Cu at (155.2, 46.5)
- added REF**: MountingHole_4.3mm_M4, Mounting_Holes:MountingHole_4.3mm_M4, F.Cu at (157.9, 139.2)
- M2, M4, M6, R10: moved to F.Cu
- moved J2 104.3 mm to (193.8, 142.4), turned to 180 degrees
- moved C7 69.0 mm to (189.6, 117.3), turned to 0 degrees
- moved M4 41.7 mm to (210.4, 78.9), turned to 180 degrees
- moved M6 41.4 mm to (210.3, 105.9), turned to 90 degrees
- moved J5 38.9 mm to (243.5, 81.0)
- moved C8 37.3 mm to (189.2, 44.7), turned to 0 degrees
- moved M2 36.2 mm to (209.9, 58.8), turned to 180 degrees
- moved R10 30.9 mm to (214.4, 91.1)
- moved R5 24.0 mm to (214.1, 68.8)
- moved M5 22.3 mm to (186.6, 102.6)
- moved M3 18.9 mm to (186.6, 78.9)
- moved R13 17.0 mm to (165.5, 112.9), turned to 180 degrees
- moved D11 14.9 mm to (165.7, 117.6), turned to 0 degrees
- moved M1 14.3 mm to (186.7, 58.9)
- moved D12 12.3 mm to (159.1, 129.2), turned to 0 degrees
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Routing:
- net /GND: track 0.00 -> 614.7 mm, vias 0 -> 64
- net /5v: track 0.00 -> 238.2 mm, vias 0 -> 5
- net /GateDriver/+12V: track 0.00 -> 177.0 mm, vias 0 -> 5
- net /GateDriver/PhaseA: track 0.00 -> 176.5 mm, vias 0 -> 23
- net /GateDriver/PhaseC: track 0.00 -> 175.7 mm, vias 0 -> 18
- net /GateDriver/PhaseB: track 0.00 -> 170.1 mm, vias 0 -> 18
- net /48v: track 0.00 -> 126.6 mm, vias 0 -> 4
- net Net-(D6-Pad2): track 0.00 -> 97.8 mm, vias 0 -> 2
- net Net-(D2-Pad2): track 0.00 -> 92.4 mm, vias 0 -> 2
- net Net-(D3-Pad2): track 0.00 -> 88.3 mm, vias 0 -> 3
- net Net-(D10-Pad2): track 0.00 -> 85.5 mm, vias 0 -> 2
- net Net-(D7-Pad2): track 0.00 -> 77.4 mm, vias 0 -> 7
- net /Microcontroller/USART_RX: track 0.00 -> 72.6 mm, vias 0 -> 1
- net /Microcontroller/USART_TX: track 0.00 -> 64.8 mm, vias 0 -> 1
- net /Microcontroller/I2C_SCL: track 0.00 -> 62.2 mm, vias 0 -> 1
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- added copper zone on B.Cu, net /48v
- added copper zone on F.Cu, net /48v
- added copper zone on B.Cu, net /5v
- added copper zone on B.Cu, net /GND
- added copper zone on F.Cu, net /GND
- added copper zone on B.Cu, net /GateDriver/PhaseA
- added copper zone on F.Cu, net /GateDriver/PhaseA
- added copper zone on B.Cu, net /GateDriver/PhaseB
- added copper zone on F.Cu, net /GateDriver/PhaseB
- added copper zone on B.Cu, net /GateDriver/PhaseC
- added copper zone on F.Cu, net /GateDriver/PhaseC
- added copper zone on F.Cu, net Net-(D1-Pad2)
- added copper zone on F.Cu, net Net-(D3-Pad2)
- added copper zone on F.Cu, net Net-(D5-Pad2)
- added copper zone on F.Cu, net Net-(D7-Pad2)
Other:
- board size 135.4 x 108.3 mm -> 178.1 x 108.3 mm
- net class HeavyDutyDefault added: clearance 0.2, trace_width 1, via_dia 1.4, via_drill 1
- net class LowDutyDefault added: clearance 0.2, trace_width 0.5, via_dia 0.8, via_drill 0.6

Commit message: updated board layout
Routing:
- net /GND: track 614.7 -> 569.9 mm
- net /GateDriver/PhaseB: track 170.1 -> 156.5 mm
- net Net-(5vConverter1-Pad2): track 34.5 -> 29.4 mm
Other:
- board text added: "Alex Simon BLDC Motor Controller 2/1/19 Rev 1"
Changed lines of the file:
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@@
     (area 72.336999 37.269 251.535001 149.325001)
     (thickness 1.6)
-    (drawings 8)
-    (tracks 901)
+    (drawings 9)
+    (tracks 889)
     (zones 0)
     (modules 67)
@@
   (layers
     (0 F.Cu signal)
-    (31 B.Cu signal)
+    (31 B.Cu signal hide)
     (32 B.Adhes user hide)
     (33 F.Adhes user hide)
@@
     (pad 1 np_thru_hole circle (at 0 0) (size 4.3 4.3) (drill 4.3) (layers *.Cu *.Mask))
   )
+  (gr_text "Alex Simon\nBLDC Motor Controller\n2/1/19\nRev 1" (at 235.204 116.332) (layer F.Mask)
+    (effects (font (size 1.5 1.5) (thickness 0.3)))
+  )
   (gr_line (start 157.861 139.192) (end 157.861 149.225) (angle 90) (layer Eco1.User) (width 0.2))
   (gr_line (start 251.46 37.846) (end 208.788 37.846) (angle 90) (layer Edge.Cuts) (width 0.15))
@@
   (segment (start 183.188 78.867) (end 192.338 78.867) (width 1) (layer F.Cu) (net 1))
   (segment (start 121.002 53.623) (end 120.59 53.623) (width 0.5) (layer F.Cu) (net 1))
-  (segment (start 118.999 66.929) (end 121.031 68.961) (width 0.5) (layer F.Cu) (net 2))
-  (segment (start 121.92 69.85) (end 122.555 70.485) (width 0.5) (layer F.Cu) (net 2))
-  (segment (start 121.031 68.961) (end 121.92 69.85) (width 0.5) (layer F.Cu) (net 2))
   (segment (start 120.59 55.323) (end 117.016 55.323) (width 0.5) (layer F.Cu) (net 2))
   (segment (start 118.999 66.929) (end 122.806 66.929) (width 0.5) (layer F.Cu) (net 2))
@@
   (segment (start 134.112 80.645) (end 132.08 80.645) (width 0.25) (layer B.Cu) (net 3))
   (segment (start 132.08 80.645) (end 132.08 84.709) (width 0.25) (layer B.Cu) (net 3))
-  (segment (start 132.08 84.709) (end 133.096 85.725) (width 0.25) (layer B.Cu) (net 3))
   (segment (start 133.096 85.725) (end 134.112 85.725) (width 0.25) (layer B.Cu) (net 3))
   (segment (start 83.312 141.605) (end 88.392 141.605) (width 0.25) (layer B.Cu) (net 3))
@@
   (segment (start 129.413 76.073) (end 129.413 73.787) (width 0.25) (layer F.Cu) (net 3))
   (segment (start 132.08 84.709) (end 132.08 80.772) (width 0.25) (layer B.Cu) (net 3))
-  (segment (start 133.096 85.725) (end 132.08 84.709) (width 0.25) (layer B.Cu) (net 3))
   (segment (start 134.112 85.725) (end 133.096 85.725) (width 0.25) (layer B.Cu) (net 3))
   (segment (start 129.862 80.645) (end 134.112 80.645) (width 0.25) (layer B.Cu) (net 3))
@@
   (segment (start 125.733 70.107) (end 129.413 73.787) (width 0.25) (layer F.Cu) (net 3))
   (segment (start 143.967 73.787) (end 144.094 73.914) (width 0.25) (layer F.Cu) (net 3))
-  (segment (start 129.74 57.023) (end 129.74 63.049) (width 0.25) (layer F.Cu) (net 3))
-  (segment (start 129.74 63.049) (end 125.733 67.056) (width 0.25) (layer F.Cu) (net 3))
   (segment (start 111.697 115.697) (end 106.553 115.697) (width 0.25) (layer F.Cu) (net 3))
   (segment (start 105.156 117.094) (end 101.221 117.094) (width 0.25) (layer F.Cu) (net 3))
@@
   (segment (start 83.312 56.007) (end 84.836 57.531) (width 0.25) (layer F.Cu) (net 3))
   (segment (start 98.86 57.531) (end 100.076 56.315) (width 0.25) (layer F.Cu) (net 3))
-  (segment (start 120.59 60.423) (end 126.34 60.423) (width 0.25) (layer F.Cu) (net 3))
   (segment (start 126.34 60.423) (end 129.74 57.023) (width 0.25) (layer F.Cu) (net 3))
   (segment (start 100.076 65.465) (end 100.076 56.315) (width 0.25) (layer F.Cu) (net 3))
   (segment (start 100.076 56.315) (end 103.476 59.715) (width 0.25) (layer F.Cu) (net 3))
   (segment (start 103.476 59.715) (end 103.476 65.465) (width 0.25) (layer F.Cu) (net 3))
-  (segment (start 100.076 56.315) (end 114.692 56.315) (width 0.25) (layer F.Cu) (net 3))
-  (segment (start 114.692 56.315) (end 115.189 56.812) (width 0.25) (layer F.Cu) (net 3))
-  (segment (start 120.59 57.023) (end 129.74 57.023) (width 0.25) (layer F.Cu) (net 3))
   (segment (start 115.189 56.812) (end 120.379 56.812) (width 0.25) (layer F.Cu) (net 3))
   (segment (start 120.379 56.812) (end 120.59 57.023) (width 0.25) (layer F.Cu) (net 3))
@@
   (segment (start 155.702 97.155) (end 154.833 96.286) (width 0.5) (layer B.Cu) (net 8))
   (segment (start 155.321 111.125) (end 155.702 110.744) (width 0.5) (layer B.Cu) (net 8))
-  (segment (start 155.702 110.744) (end 155.702 97.155) (width 0.5) (layer B.Cu) (net 8))
   (segment (start 148.768 96.266) (end 151.13 96.266) (width 0.5) (layer F.Cu) (net 8))
   (segment (start 151.15 96.286) (end 153.416 96.286) (width 0.5) (layer B.Cu) (net 8))
@@
   )
   (zone (net 3) (net_name /GND) (layer F.Cu) (hatch edge 0.508)
-    (connect_pads (clearance 0.35))
+    (connect_pads yes (clearance 0.35))
     (min_thickness 0.35)
     (fill yes (arc_segments 16) (thermal_gap 0.65) (thermal_bridge_width 0.4))
