File: hardware/bldc_v1.sch (KiCad schematic (older format))
At the start: 5 parts, among them J1 Conn_01x06, J2 1x2_ScrewTerminal_65A, J3 Screw_Terminal_01x05, J4 RJ45, J5 Screw_Terminal_01x03

Commit message: layed parts out on board
Changed lines of the file:
@@
 LIBS:crf_1
 LIBS:STM32F4-DISCOVERY-SIMON
+LIBS:bldc_v1-cache
 EELAYER 25 0
 EELAYER END
@@
 Wire Wire Line
 	1650 1050 1400 1050
-Wire Wire Line
-	7450 4550 7450 3950
-Connection ~ 7450 3950
-Wire Wire Line
-	7350 4550 7350 3850
-Connection ~ 7350 3850
-Wire Wire Line
-	7250 4550 7250 3750
-Connection ~ 7250 3750
 $Comp
 L Conn_01x06 J1
@@
 NoConn ~ 4400 4450
 NoConn ~ 4300 4450
+Wire Wire Line
+	7250 4550 7250 3950
+Connection ~ 7250 3950
+Wire Wire Line
+	7350 4550 7350 3850
+Connection ~ 7350 3850
+Wire Wire Line
+	7450 4550 7450 3750
+Connection ~ 7450 3750
 $EndSCHEMATC

Commit message: updated part numbers
Connections:
- wire segments 59 -> 61
Changed lines of the file:
@@
 LIBS:crf_1
 LIBS:STM32F4-DISCOVERY-SIMON
+LIBS:bldc_v1-cache
 EELAYER 25 0
 EELAYER END
@@
 F0 "GateDriver" 60
 F1 "GateDriver.sch" 60
-F2 "PhaseA" I R 6650 3750 60
-F3 "PhaseB" I R 6650 3850 60
-F4 "PhaseC" I R 6650 3950 60
-F5 "GND" U L 4900 2800 60
-F6 "LS_A_GATE" O R 6650 3100 60
-F7 "HS_A_GATE" O R 6650 3000 60
-F8 "LS_B_GATE" O R 6650 3300 60
-F9 "HS_B_GATE" O R 6650 3200 60
-F10 "LS_C_GATE" O R 6650 3500 60
-F11 "HS_C_GATE" O R 6650 3400 60
-F12 "LS_A_TTL_PWM" I L 4900 3100 60
-F13 "HS_A_TTL_PWM" I L 4900 3000 60
-F14 "LS_B_TTL_PWM" I L 4900 3300 60
-F15 "HS_B_TTL_PWM" I L 4900 3200 60
-F16 "LS_C_TTL_PWM" I L 4900 3500 60
-F17 "HS_C_TTL_PWM" I L 4900 3400 60
-F18 "+12V" I L 4900 2700 60
+F2 "PhaseC" I R 6650 4150 60
+F3 "GND" U L 4900 2800 60
+F4 "LS_A_GATE" O R 6650 3100 60
+F5 "HS_A_GATE" O R 6650 3000 60
+F6 "LS_B_GATE" O R 6650 3300 60
+F7 "HS_B_GATE" O R 6650 3200 60
+F8 "LS_C_GATE" O R 6650 3500 60
+F9 "HS_C_GATE" O R 6650 3400 60
+F10 "LS_A_TTL_PWM" I L 4900 3100 60
+F11 "HS_A_TTL_PWM" I L 4900 3000 60
+F12 "LS_B_TTL_PWM" I L 4900 3300 60
+F13 "HS_B_TTL_PWM" I L 4900 3200 60
+F14 "LS_C_TTL_PWM" I L 4900 3500 60
+F15 "HS_C_TTL_PWM" I L 4900 3400 60
+F16 "+12V" I L 4900 2700 60
+F17 "PhaseADrain" I R 6650 3700 60
+F18 "PhaseBDrain" I R 6650 3800 60
 $EndSheet
 $Sheet
@@
 F0 "MOSFETS" 60
 F1 "MOSFETS.sch" 60
-F2 "PhaseA" O L 7900 3750 60
-F3 "PhaseB" O L 7900 3850 60
-F4 "PhaseC" O L 7900 3950 60
+F2 "PhaseA" O L 7900 3950 60
+F3 "PhaseB" O L 7900 4050 60
+F4 "PhaseC" O L 7900 4150 60
 F5 "GND" U L 7900 2850 60
 F6 "HS_A_GATE" I L 7900 3000 60
@@
 F14 "48v" I L 7900 2650 60
 F15 "5V" I L 7900 2750 60
+F16 "PhaseADrain" O L 7900 3700 60
+F17 "PhaseBDrain" O L 7900 3800 60
 $EndSheet
 Wire Wire Line
@@
 	7750 2850 7900 2850
 Wire Wire Line
-	6650 3950 7900 3950
-Wire Wire Line
-	6650 3750 7900 3750
-Wire Wire Line
-	6650 3850 7900 3850
-Wire Wire Line
 	4800 2800 4900 2800
 Text Label 9600 2700 0    60   ~ 0
@@
 NoConn ~ 4300 4450
 Wire Wire Line
-	7250 4550 7250 3950
-Connection ~ 7250 3950
-Wire Wire Line
-	7350 4550 7350 3850
-Connection ~ 7350 3850
-Wire Wire Line
-	7450 4550 7450 3750
-Connection ~ 7450 3750
+	7900 4150 6650 4150
+Wire Wire Line
+	7250 4550 7250 4150
+Connection ~ 7250 4150
+Wire Wire Line
+	7900 3700 6650 3700
+Wire Wire Line
+	7900 3800 6650 3800
+Wire Wire Line
+	7900 3950 7450 3950
+Wire Wire Line
+	7450 3950 7450 4550
+Wire Wire Line
+	7900 4050 7350 4050
+Wire Wire Line
+	7350 4050 7350 4550
 $EndSCHEMATC

Commit message: Converted to kicad 5
Parts:
- J1: symbol Conn_01x06 -> Connector_Generic:Conn_01x06
- J2: symbol 1x2_ScrewTerminal_65A -> infineon:1x2_ScrewTerminal_65A
- J3: symbol Screw_Terminal_01x05 -> Connector:Screw_Terminal_01x05
- J4: symbol RJ45 -> Connector:RJ45
- J5: symbol Screw_Terminal_01x03 -> Connector:Screw_Terminal_01x03
Connections:
- wire segments 61 -> 64
Changed lines of the file:
@@
-EESchema Schematic File Version 2
-LIBS:power
-LIBS:device
-LIBS:switches
-LIBS:relays
-LIBS:motors
-LIBS:transistors
-LIBS:conn
-LIBS:linear
-LIBS:regul
-LIBS:74xx
-LIBS:cmos4000
-LIBS:adc-dac
-LIBS:memory
-LIBS:xilinx
-LIBS:microcontrollers
-LIBS:dsp
-LIBS:microchip
-LIBS:analog_switches
-LIBS:motorola
-LIBS:texas
-LIBS:intel
-LIBS:audio
-LIBS:interface
-LIBS:digital-audio
-LIBS:philips
-LIBS:display
-LIBS:cypress
-LIBS:siliconi
-LIBS:opto
-LIBS:atmel
-LIBS:contrib
-LIBS:valves
-LIBS:infineon
-LIBS:crf_1
-LIBS:STM32F4-DISCOVERY-SIMON
-LIBS:bldc_v1-cache
-EELAYER 25 0
+EESchema Schematic File Version 4
+EELAYER 26 0
 EELAYER END
 $Descr A4 11693 8268
@@
 F0 "GateDriver" 60
 F1 "GateDriver.sch" 60
-F2 "PhaseC" I R 6650 4150 60
-F3 "GND" U L 4900 2800 60
-F4 "LS_A_GATE" O R 6650 3100 60
-F5 "HS_A_GATE" O R 6650 3000 60
-F6 "LS_B_GATE" O R 6650 3300 60
-F7 "HS_B_GATE" O R 6650 3200 60
-F8 "LS_C_GATE" O R 6650 3500 60
-F9 "HS_C_GATE" O R 6650 3400 60
-F10 "LS_A_TTL_PWM" I L 4900 3100 60
-F11 "HS_A_TTL_PWM" I L 4900 3000 60
-F12 "LS_B_TTL_PWM" I L 4900 3300 60
-F13 "HS_B_TTL_PWM" I L 4900 3200 60
-F14 "LS_C_TTL_PWM" I L 4900 3500 60
-F15 "HS_C_TTL_PWM" I L 4900 3400 60
-F16 "+12V" I L 4900 2700 60
-F17 "PhaseADrain" I R 6650 3700 60
-F18 "PhaseBDrain" I R 6650 3800 60
+F2 "GND" U L 4900 2800 60
+F3 "LS_A_GATE" O R 6650 3100 60
+F4 "HS_A_GATE" O R 6650 3000 60
+F5 "LS_B_GATE" O R 6650 3300 60
+F6 "HS_B_GATE" O R 6650 3200 60
+F7 "LS_C_GATE" O R 6650 3500 60
+F8 "HS_C_GATE" O R 6650 3400 60
+F9 "LS_A_TTL_PWM" I L 4900 3100 60
+F10 "HS_A_TTL_PWM" I L 4900 3000 60
+F11 "LS_B_TTL_PWM" I L 4900 3300 60
+F12 "HS_B_TTL_PWM" I L 4900 3200 60
+F13 "LS_C_TTL_PWM" I L 4900 3500 60
+F14 "HS_C_TTL_PWM" I L 4900 3400 60
+F15 "+12V" I L 4900 2700 60
+F16 "PhaseASource" I R 6650 3700 60
+F17 "PhaseBSource" I R 6650 3800 60
+F18 "PhaseCSource" I R 6650 4150 60
 $EndSheet
 $Sheet
@@
 F14 "48v" I L 7900 2650 60
 F15 "5V" I L 7900 2750 60
-F16 "PhaseADrain" O L 7900 3700 60
-F17 "PhaseBDrain" O L 7900 3800 60
+F16 "PhaseASource" O L 7900 3700 60
+F17 "PhaseBSource" O L 7900 3800 60
 $EndSheet
 Wire Wire Line
@@
 $EndSheet
 Wire Wire Line
-	4300 2100 7400 2100
+	4300 2100 4750 2100
 Wire Wire Line
 	4900 2700 4700 2700
@@
 	4700 2300 4300 2300
 Wire Wire Line
-	3350 1750 7500 1750
+	3350 1750 3500 1750
 Wire Wire Line
 	3500 1750 3500 2100
@@
 	1650 1050 1400 1050
 $Comp
-L Conn_01x06 J1
+L Connector_Generic:Conn_01x06 J1
 U 1 1 5AB8F4C0
 P 1050 3500
@@
 $EndComp
 $Comp
-L Screw_Terminal_01x05 J3
+L Connector:Screw_Terminal_01x05 J3
 U 1 1 5AB91720
 P 1900 2300
@@
 	2000 2600 2000 2500
 $Comp
-L 1x2_ScrewTerminal_65A J2
+L infineon:1x2_ScrewTerminal_65A J2
 U 1 1 5ABA8578
 P 1200 1050
@@
 $EndComp
 $Comp
-L Screw_Terminal_01x03 J5
+L Connector:Screw_Terminal_01x03 J5
 U 1 1 5ABABEF7
 P 7350 4750
@@
 	0    1    1    0
 $EndComp
-$Comp
-L RJ45 J4
-U 1 1 5ABC4D57
-P 4350 4900
-F 0 "J4" H 4550 5400 50  0000 C CNN
-F 1 "RJ45" H 4200 5400 50  0000 C CNN
-F 2 "Connectors:RJ45_8" H 4350 4900 50  0001 C CNN
-F 3 "" H 4350 4900 50  0001 C CNN
-F 4 "SS-6488S-A-NF" H 4350 5500 60  0000 C CNN "PN"
-	1    4350 4900
-	-1   0    0    1
-$EndComp
 Wire Wire Line
 	4200 4200 4200 4450
@@
 NoConn ~ 4300 4450
 Wire Wire Line
-	7900 4150 6650 4150
+	7900 4150 7250 4150
 Wire Wire Line
 	7250 4550 7250 4150
@@
 Wire Wire Line
 	7350 4050 7350 4550
+Wire Wire Line
+	4750 2100 7400 2100
+Wire Wire Line
+	3500 1750 7500 1750
+Wire Wire Line
+	7250 4150 6650 4150
+$Comp
+L Connector:RJ45 J4
+U 1 1 5ABC4D57
+P 4400 4850
+F 0 "J4" V 4050 5100 50  0000 C CNN
+F 1 "RJ45" V 4050 4700 50  0000 C CNN
+F 2 "Connectors:RJ45_8" H 4400 4850 50  0001 C CNN
+F 3 "" H 4400 4850 50  0001 C CNN
+F 4 "SS-6488S-A-NF" V 3950 4900 60  0000 C CNN "PN"
+	1    4400 4850
+	0    -1   -1   0
+$EndComp
 $EndSCHEMATC
