File: hardware/bldc_v1.sch (KiCad schematic (older format))
At the start: 5 parts, among them J1 Conn_01x06, J2 1x2_ScrewTerminal_65A, J3 Screw_Terminal_01x05, J4 RJ45, J5 Screw_Terminal_01x03

Commit message: Updated schematic for additional capacitors
Parts:
- added C17: 330uF, symbol Device:CP1
Connections:
- wire segments 64 -> 72
Changed lines of the file:
@@
 48v
 Connection ~ 3500 1750
-Text Label 1650 950  0    60   ~ 0
+Text Label 2350 750  0    60   ~ 0
 48v
-Wire Wire Line
-	1650 950  1400 950
-Text Label 1650 1050 0    60   ~ 0
+Text Label 2350 1250 0    60   ~ 0
 GND
-Wire Wire Line
-	1650 1050 1400 1050
 $Comp
 L Connector_Generic:Conn_01x06 J1
@@
 	0    -1   -1   0
 $EndComp
+$Comp
+L Device:CP1 C17
+U 1 1 5C5C16E0
+P 1900 1000
+F 0 "C17" H 2015 1091 50  0000 L CNN
+F 1 "330uF" H 2015 1000 50  0000 L CNN
+F 2 "" H 1900 1000 50  0001 C CNN
+F 3 "~" H 1900 1000 50  0001 C CNN
+F 4 "EEV-TG2A331M " H 2015 909 50  0000 L CNN "PN"
+	1    1900 1000
+	1    0    0    -1
+$EndComp
+Wire Wire Line
+	2350 1250 1900 1250
+Wire Wire Line
+	1900 1250 1900 1150
+Wire Wire Line
+	1900 850  1900 750
+Wire Wire Line
+	1900 750  2350 750
+Wire Wire Line
+	1750 950  1750 750
+Wire Wire Line
+	1750 750  1900 750
+Wire Wire Line
+	1400 950  1750 950
+Connection ~ 1900 750
+Wire Wire Line
+	1750 1050 1750 1250
+Wire Wire Line
+	1750 1250 1900 1250
+Wire Wire Line
+	1400 1050 1750 1050
+Connection ~ 1900 1250
 $EndSCHEMATC

Commit message: Added additional capacitors for 48v bus
Parts:
- added C18, C19: 100u, Capacitors_SMD:CP_Elec_10x10, symbol Device:CP1
- C17: value 330uF -> 100u; footprint (none) -> Capacitors_SMD:CP_Elec_10x10; PN EEV-TG2A331M -> EEE-1JA101P
Connections:
- wire segments 72 -> 80
Changed lines of the file:
@@
 48v
 Connection ~ 3500 1750
-Text Label 2350 750  0    60   ~ 0
+Text Label 3450 700  0    60   ~ 0
 48v
-Text Label 2350 1250 0    60   ~ 0
+Text Label 3450 1250 0    60   ~ 0
 GND
 $Comp
@@
 L Device:CP1 C17
 U 1 1 5C5C16E0
-P 1900 1000
-F 0 "C17" H 2015 1091 50  0000 L CNN
-F 1 "330uF" H 2015 1000 50  0000 L CNN
-F 2 "" H 1900 1000 50  0001 C CNN
-F 3 "~" H 1900 1000 50  0001 C CNN
-F 4 "EEV-TG2A331M " H 2015 909 50  0000 L CNN "PN"
-	1    1900 1000
+P 1950 1000
+F 0 "C17" H 2065 1091 50  0000 L CNN
+F 1 "100u" H 2065 1000 50  0000 L CNN
+F 2 "Capacitors_SMD:CP_Elec_10x10" H 1950 1000 50  0001 C CNN
+F 3 "~" H 1950 1000 50  0001 C CNN
+F 4 "EEE-1JA101P" V 1800 750 50  0000 L CNN "PN"
+	1    1950 1000
 	1    0    0    -1
 $EndComp
 Wire Wire Line
-	2350 1250 1900 1250
-Wire Wire Line
-	1900 1250 1900 1150
-Wire Wire Line
-	1900 850  1900 750
-Wire Wire Line
-	1900 750  2350 750
-Wire Wire Line
-	1750 950  1750 750
-Wire Wire Line
-	1750 750  1900 750
-Wire Wire Line
 	1400 950  1750 950
-Connection ~ 1900 750
 Wire Wire Line
 	1750 1050 1750 1250
 Wire Wire Line
-	1750 1250 1900 1250
-Wire Wire Line
 	1400 1050 1750 1050
-Connection ~ 1900 1250
+Wire Wire Line
+	1750 1250 1950 1250
+Wire Wire Line
+	1950 1150 1950 1250
+Connection ~ 1950 1250
+Wire Wire Line
+	1950 850  1950 700
+Wire Wire Line
+	1950 700  1750 700
+Wire Wire Line
+	1750 700  1750 950
+$Comp
+L Device:CP1 C18
+U 1 1 5C53255D
+P 2500 1000
+F 0 "C18" H 2615 1091 50  0000 L CNN
+F 1 "100u" H 2615 1000 50  0000 L CNN
+F 2 "Capacitors_SMD:CP_Elec_10x10" H 2500 1000 50  0001 C CNN
+F 3 "~" H 2500 1000 50  0001 C CNN
+F 4 "EEE-1JA101P" V 2350 750 50  0000 L CNN "PN"
+	1    2500 1000
+	1    0    0    -1
+$EndComp
+$Comp
+L Device:CP1 C19
+U 1 1 5C53258F
+P 3050 1000
+F 0 "C19" H 3165 1091 50  0000 L CNN
+F 1 "100u" H 3165 1000 50  0000 L CNN
+F 2 "Capacitors_SMD:CP_Elec_10x10" H 3050 1000 50  0001 C CNN
+F 3 "~" H 3050 1000 50  0001 C CNN
+F 4 "EEE-1JA101P" V 2900 750 50  0000 L CNN "PN"
+	1    3050 1000
+	1    0    0    -1
+$EndComp
+Wire Wire Line
+	3050 1250 3050 1150
+Wire Wire Line
+	1950 1250 2500 1250
+Wire Wire Line
+	2500 1150 2500 1250
+Connection ~ 2500 1250
+Wire Wire Line
+	2500 1250 3050 1250
+Wire Wire Line
+	2500 850  2500 700
+Wire Wire Line
+	2500 700  1950 700
+Connection ~ 1950 700
+Wire Wire Line
+	3050 850  3050 700
+Wire Wire Line
+	3050 700  2500 700
+Connection ~ 2500 700
+Wire Wire Line
+	3450 700  3050 700
+Connection ~ 3050 700
+Wire Wire Line
+	3050 1250 3450 1250
+Connection ~ 3050 1250
 $EndSCHEMATC

Commit message: completely restarted
Parts:
- removed C17, C18, C19: 100u, Capacitors_SMD:CP_Elec_10x10, symbol Device:CP1
- removed J1: Conn_01x06, Pin_Headers:Pin_Header_Straight_1x06_Pitch2.54mm_SMD_Pin1Right, symbol Connector_Generic:Conn_01x06
- removed J2: 1x2_ScrewTerminal_65A, custom:1x2_ScrewTerminal_65A, symbol infineon:1x2_ScrewTerminal_65A
- removed J3: Screw_Terminal_01x05, custom:1x5_ScrewTerminal_1A, symbol Connector:Screw_Terminal_01x05
- removed J4: RJ45, Connectors:RJ45_8, symbol Connector:RJ45
- removed J5: Screw_Terminal_01x03, custom:1x3_ScrewTerminal_65A, symbol Connector:Screw_Terminal_01x03
- added C1, C2, C3: 1mF, symbol Device:CP1_Small
- added J1: Screw_Terminal_01x02, symbol Connector:Screw_Terminal_01x02
- added J2: Conn_02x07_Counter_Clockwise, symbol Connector_Generic:Conn_02x07_Counter_Clockwise
- added J3: Screw_Terminal_01x03, symbol Connector:Screw_Terminal_01x03
Connections:
- net labels added: 12v, HS_A_TTL_PWM, HS_B_TTL_PWM, HS_C_TTL_PWM, LS_A_TTL_PWM, LS_B_TTL_PWM, LS_C_TTL_PWM, PHASEA_FB, PHASEB_FB, PHASE_A, PHASE_B, PHASE_C
- net labels removed: FB_A, FB_B
- wire segments 80 -> 58
- no-connect marks 8 -> 2
Other:
- note removed: "Intentionally connected \nbackwards"
