File: hardware/Operator/Operator.kicad_pcb (KiCad board)
At the start: 2 copper layers, 9 parts, among them J1 RJ45, J2 Screw_Terminal_01x02, U1 DS89C21

Commit message: Added gerber files
Parts:
- added J3: Conn_01x06_Male, Connector_PinHeader_2.54mm:PinHeader_1x06_P2.54mm_Vertical, F.Cu at (139.7, 79.9)
- moved R3 39.6 mm to (171.8, 59.7), turned to 180 degrees
- moved R2 27.4 mm to (145.5, 83.4)
- moved R1 23.9 mm to (145.5, 88.9)
- moved C2 23.6 mm to (164.5, 72.8), turned to 90 degrees
- moved U1 16.4 mm to (154.2, 86.9), turned to 180 degrees
- moved C1 7.10 mm to (148.3, 72.8), turned to 90 degrees
- moved J2 3.43 mm to (183.3, 68.7)
Connections:
- A1 pad 13: (no net) -> /A4
- A1 pad 14: (no net) -> /A5
- A1 pad 18: (no net) -> /D3
- A1 pad 20: (no net) -> /D5
Routing:
- net /5v: track 0.00 -> 115.0 mm
- net /A5: track 0.00 -> 60.5 mm
- net /A4: track 0.00 -> 54.8 mm
- net /D3: track 0.00 -> 39.6 mm
- net /D5: track 0.00 -> 35.5 mm
- net /USART_RX: track 0.00 -> 32.1 mm, vias 0 -> 1
- net /-RX: track 0.00 -> 30.6 mm
- net /USART_TX: track 0.00 -> 30.1 mm, vias 0 -> 1
- net /+Tx: track 0.00 -> 29.6 mm
- net /-TX: track 0.00 -> 27.3 mm
- net /+RX: track 0.00 -> 26.5 mm
- net /A0: track 0.00 -> 19.3 mm
- net /TransEnable_TTL: track 0.00 -> 17.1 mm
- net /GND: track 0.00 -> 2.41 mm, vias 0 -> 2
- added copper zone on B.Cu, net /GND
- added copper zone on F.Cu, net /GND
Other:
- board outline added: 53.8 x 54.2 mm
- net class Default: trace_width 0.25 -> 0.5; via_dia 0.8 -> 0.9; via_drill 0.4 -> 0.5
